File: th-vco-1/kicad_files/vco-1.sch (KiCad schematic (older format))
At the start: 69 parts, among them J1 PWM, J2 1V/OCT, J3 EXP FM, J4 LIN FM, J5 EURORACK POWER, J6 PULSE, J7 SINE, J8 TRIANGLE, Q1 2N3906, Q2 2N3906, Q3 2N3904, Q4 2N3904, Q5 2N3904, Q6 2N3904, U1 TL072, U2 CA3080, U3 TL072, U4 TL072

Commit message: Changed resistor values to 12 V
Changed most of the resistors mentioned in these threads:
http://www.electro-music.com/forum/topic-54360.html
http://electro-music.com/forum/topic-36820.html

Not yet changed R23 or R41, in the original schematics. Will do
that after trying it in real life.
Also maybe R46, for fine tuning to span one octave.

Added bill of materials (obviously with the above unchanged values,
that will probably change).
Parts:
- R20: value 20k -> 24k
- R26: value 100k -> 110k
- R28: value 5.1k -> 3.9k
- R30, R33: value 12k -> 14k
- R35: value 3k -> 2k
- R36: value 1.8k -> 2k
- R6: value 1.5M -> 1.2M
- R8: value 2k -> 2k +3500ppm/C thermistor
Other:
- note added: "NOTE: Forgot to change values for 12V before making PCB rev A. \nHave not tested yet, but the changed resistors are: \nR6, R20, R28, R26, R30, R33, R35, R36.\nPossibly also R11 should be changed, to 18k.\nFor pulse width adj., maybe change R15 (to 256k).\nSee http://www.electro-music.com/forum/topic-54360.html and\nhttp://electro-music.com/forum/topic-36820.html"
- note added: "NOTE: R8 should ideally be a +3500ppm/C 2K thermistor (tempco), \nand Q1/Q2 should be mechanically bonded (e.g. by epoxy).\nFor best result, R8 should also be physically bonded to Q1/Q2."
- note removed: "NOTE: R8 should ideally be a +3500ppm/Co 2K thermistor (tempco), \nand Q1/Q2 should be mechanically bonded (e.g. by epoxy).\nFor best result, R8 should also be physically bonded to Q1/Q2."
Changed lines of the file:
@@
 P 2600 1750
 F 0 "R8" V 2680 1750 50  0000 C CNN
-F 1 "2k" V 2600 1750 50  0000 C CNN
+F 1 "2k +3500ppm/C thermistor" V 2500 1750 50  0000 C CNN
 F 2 "Resistors_THT:R_Axial_DIN0309_L9.0mm_D3.2mm_P12.70mm_Horizontal" V 2530 1750 50  0001 C CNN
 F 3 "" H 2600 1750 50  0001 C CNN
@@
 P 2350 4200
 F 0 "R6" V 2430 4200 50  0000 C CNN
-F 1 "1.5M" V 2350 4200 50  0000 C CNN
+F 1 "1.2M" V 2350 4200 50  0000 C CNN
 F 2 "Resistors_THT:R_Axial_DIN0309_L9.0mm_D3.2mm_P12.70mm_Horizontal" V 2280 4200 50  0001 C CNN
 F 3 "" H 2350 4200 50  0001 C CNN
@@
 P 7150 4800
 F 0 "R20" V 7230 4800 50  0000 C CNN
-F 1 "20k" V 7150 4800 50  0000 C CNN
+F 1 "24k" V 7150 4800 50  0000 C CNN
 F 2 "Resistors_THT:R_Axial_DIN0309_L9.0mm_D3.2mm_P12.70mm_Horizontal" V 7080 4800 50  0001 C CNN
 F 3 "" H 7150 4800 50  0001 C CNN
@@
 P 7950 4800
 F 0 "R28" V 8030 4800 50  0000 C CNN
-F 1 "5.1k" V 7950 4800 50  0000 C CNN
+F 1 "3.9k" V 7950 4800 50  0000 C CNN
 F 2 "Resistors_THT:R_Axial_DIN0309_L9.0mm_D3.2mm_P12.70mm_Horizontal" V 7880 4800 50  0001 C CNN
 F 3 "" H 7950 4800 50  0001 C CNN
@@
 P 7650 6000
 F 0 "R26" V 7730 6000 50  0000 C CNN
-F 1 "100k" V 7650 6000 50  0000 C CNN
+F 1 "110k" V 7650 6000 50  0000 C CNN
 F 2 "Resistors_THT:R_Axial_DIN0309_L9.0mm_D3.2mm_P12.70mm_Horizontal" V 7580 6000 50  0001 C CNN
 F 3 "" H 7650 6000 50  0001 C CNN
@@
 P 8350 2250
 F 0 "R30" V 8430 2250 50  0000 C CNN
-F 1 "12k" V 8350 2250 50  0000 C CNN
+F 1 "14k" V 8350 2250 50  0000 C CNN
 F 2 "Resistors_THT:R_Axial_DIN0309_L9.0mm_D3.2mm_P12.70mm_Horizontal" V 8280 2250 50  0001 C CNN
 F 3 "" H 8350 2250 50  0001 C CNN
@@
 P 8850 3100
 F 0 "R33" V 8930 3100 50  0000 C CNN
-F 1 "12k" V 8850 3100 50  0000 C CNN
+F 1 "14k" V 8850 3100 50  0000 C CNN
 F 2 "Resistors_THT:R_Axial_DIN0309_L9.0mm_D3.2mm_P12.70mm_Horizontal" V 8780 3100 50  0001 C CNN
 F 3 "" H 8850 3100 50  0001 C CNN
@@
 P 9500 1150
 F 0 "R35" V 9580 1150 50  0000 C CNN
-F 1 "3k" V 9500 1150 50  0000 C CNN
+F 1 "2k" V 9500 1150 50  0000 C CNN
 F 2 "Resistors_THT:R_Axial_DIN0309_L9.0mm_D3.2mm_P12.70mm_Horizontal" V 9430 1150 50  0001 C CNN
 F 3 "" H 9500 1150 50  0001 C CNN
@@
 P 9800 1350
 F 0 "R36" V 9880 1350 50  0000 C CNN
-F 1 "1.8k" V 9800 1350 50  0000 C CNN
+F 1 "2k" V 9800 1350 50  0000 C CNN
 F 2 "Resistors_THT:R_Axial_DIN0309_L9.0mm_D3.2mm_P12.70mm_Horizontal" V 9730 1350 50  0001 C CNN
 F 3 "" H 9800 1350 50  0001 C CNN
@@
 Wire Wire Line
 	7150 5750 8350 5750
-Text Notes 900  7050 0    60   ~ 0
-NOTE: R8 should ideally be a +3500ppm/Co 2K thermistor (tempco), \nand Q1/Q2 should be mechanically bonded (e.g. by epoxy).\nFor best result, R8 should also be physically bonded to Q1/Q2.
+Text Notes 600  6700 0    60   ~ 0
+NOTE: R8 should ideally be a +3500ppm/C 2K thermistor (tempco), \nand Q1/Q2 should be mechanically bonded (e.g. by epoxy).\nFor best result, R8 should also be physically bonded to Q1/Q2.
+Text Notes 600  7650 0    60   ~ 0
+NOTE: Forgot to change values for 12V before making PCB rev A. \nHave not tested yet, but the changed resistors are: \nR6, R20, R28, R26, R30, R33, R35, R36.\nPossibly also R11 should be changed, to 18k.\nFor pulse width adj., maybe change R15 (to 256k).\nSee http://www.electro-music.com/forum/topic-54360.html and\nhttp://electro-music.com/forum/topic-36820.html
 $EndSCHEMATC

Commit message: Update after rev A failure
Fixed most of the errors found in rev A. No fix for the
reverse pots, though, since I don't know how.
At this point it would also mean to re-CAD, not too happy
about that.
Parts:
- added C10, C9: 10uF, Capacitors_THT:CP_Radial_D5.0mm_P2.00mm, symbol CP
- added C11, C12, C13, C14, C5, C6, C7, C8: 10nF, Capacitors_THT:C_Rect_L7.2mm_W3.5mm_P5.00mm_FKS2_FKP2_MKS2_MKP2, symbol C
- C1, C2, C4: footprint Capacitors_THT:C_Axial_L3.8mm_D2.6mm_P7.50mm_Horizontal -> Capacitors_THT:C_Rect_L7.2mm_W3.5mm_P5.00mm_FKS2_FKP2_MKS2_MKP2
- C3: value 1n -> 1n polystyrene
- R1, R2, R3: value 100 -> 100k; footprint Resistors_THT:R_Axial_DIN0309_L9.0mm_D3.2mm_P12.70mm_Horizontal -> Resistors_THT:R_Axial_DIN0207_L6.3mm_D2.5mm_P7.62mm_Horizontal
- R10, R11, R12, R13, R14, R15, R16, R17, R18, R19, R20, R21, R22, R23, R24, R25, R26, R27, R28, R29, R30, R31, R32, R33, R34, R35, R36, R4, R5, R6, R7, R9: footprint Resistors_THT:R_Axial_DIN0309_L9.0mm_D3.2mm_P12.70mm_Horizontal -> Resistors_THT:R_Axial_DIN0207_L6.3mm_D2.5mm_P7.62mm_Horizontal
- RV10, RV6, RV9: footprint Potentiometers:Potentiometer_Trimmer_Bourns_3266Y -> Potentiometers:Potentiometer_Trimmer_ACP_CA6h_Vertical
Connections:
- net +12V: now also J5.1 (Pin_1), C11.1, C13.1, C5.1, C7.1, C9.1
- net -12V: now also J5.9 (Pin_9), C10.2, C12.2, C14.2, C6.2, C8.2
- net GND: now also J5.3 (Pin_3), J5.5 (Pin_5), J5.7 (Pin_7), U1.3 (+), U1.5 (+), C10.1, C11.2, C12.1, C13.2, C14.1, C5.2, C6.1, C7.2, C8.1, C9.2; no longer U1.2 (-), U1.6 (-)
- net at R1.1, R2.1, R3.1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: now also U1.2 (-); no longer U1.3 (+)
- net at R7.1: now also C2.2, Q1.3 (C), R6.1, U1.6 (-); no longer U1.5 (+)
- no-connect marks 5 -> 0
Other:
- note added: "B"
- note added: "July 11, 2018"
- note removed: "2018-04-29"
- note removed: "A"
- moved on the sheet: C1, C3, J4, R12, R13, R30, R32, R33, R34, R35, R6, R7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

Commit message: Use 16 pole power connector
Even though a 10 pole would be enough, my current plan is
to use 16 pole for all boards, thus minimizing cost for
power connectors/cables.

Possibly a bad idea, but if I will go through with the plans
to run workshops using these boards, there will be a LOT of
component bought, and it makes sense to keep cost down.
Parts:
- J5: value EURORACK POWER -> EURO_POWER; footprint Pin_Headers:Pin_Header_Straight_2x05_Pitch2.54mm -> Pin_Headers:Pin_Header_Straight_2x08_Pitch2.54mm; symbol Conn_02x05_Odd_Even -> Conn_02x08_Odd_Even
Connections:
- net +12V: now also J5.10 (Pin_10), J5.9 (Pin_9); no longer J5.1 (Pin_1), J5.2 (Pin_2)
- net -12V: now also J5.1 (Pin_1), J5.2 (Pin_2); no longer J5.10 (Pin_10), J5.9 (Pin_9)
- no-connect marks 0 -> 6
Other:
- moved on the sheet: C10, C9
