File: passive_aggressive_lpg/kicad_files/passive_aggressive_1.sch (KiCad schematic (older format))
At the start: 18 parts, among them J1 Audio-Jack-2, J2 Audio-Jack-2, J3 Audio-Jack-2, SW1 SLEW/ATT, SW2 HIGH, SW3 LOW, U1 NSL-32SR2

Commit message: Clean up passive LPG after building the second
Parts:
- removed R2: 200, Potentiometers:Potentiometer_Trimmer_ACP_CA9h2.5_Vertical_Px2.5mm_Py5.0mm, symbol RTRIM
- added C5: 470nF, Capacitors_THT:C_Rect_L7.2mm_W3.5mm_P5.00mm_FKS2_FKP2_MKS2_MKP2, symbol C
- added C6: 68nF, Capacitors_THT:C_Rect_L7.2mm_W3.5mm_P5.00mm_FKS2_FKP2_MKS2_MKP2, symbol C
- added R2: 180, Resistors_THT:R_Axial_DIN0207_L6.3mm_D2.5mm_P7.62mm_Horizontal, symbol R
- C1, C2: value 1000u -> 1000uF
- C3: value 100n -> 100nF
- C4: value 470n -> 470nF
- J1: value Audio-Jack-2 -> AUDIO_IN; footprint Wire_Pads:SolderWirePad_3x_2mmDrill -> Pin_Headers:Pin_Header_Straight_1x02_Pitch2.54mm
- J2: value Audio-Jack-2 -> CV_IN; footprint (none) -> Pin_Headers:Pin_Header_Straight_1x02_Pitch2.54mm
- J3: value Audio-Jack-2 -> AUDIO_OUT; footprint (none) -> Pin_Headers:Pin_Header_Straight_1x02_Pitch2.54mm
- R1, R4: footprint Resistors_THT:R_Axial_DIN0207_L6.3mm_D2.5mm_P10.16mm_Horizontal -> Resistors_THT:R_Axial_DIN0207_L6.3mm_D2.5mm_P7.62mm_Horizontal
- R3: value 100 -> 1.5k; footprint Resistors_THT:R_Axial_DIN0207_L6.3mm_D2.5mm_P10.16mm_Horizontal -> Resistors_THT:R_Axial_DIN0207_L6.3mm_D2.5mm_P7.62mm_Horizontal
- SW2: value HIGH -> FILTER1; footprint Pin_Headers:Pin_Header_Straight_1x02_Pitch2.54mm -> Pin_Headers:Pin_Header_Straight_1x03_Pitch2.54mm; symbol SW_SPDT -> SW_SPDT_MSM
- SW3: value LOW -> FILTER2; footprint Pin_Headers:Pin_Header_Straight_1x02_Pitch2.54mm -> Pin_Headers:Pin_Header_Straight_1x03_Pitch2.54mm; symbol SW_SPDT -> SW_SPDT_MSM
Connections:
- net GND: now also R2.2
- net at C3.2, C4.2, J3.1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: now also C5.2, C6.2
- net at C2.1, D1.1 (K), R3.1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: now also RV1.2, SW1.1 (A); no longer SW1.3 (C)
- net at R3.2: now also RV1.3, R2.1; no longer RV1.2
- net at SW2.3: now also C5.1
- net at SW3.3: now also C6.1
- no-connect marks 3 -> 1
Other:
- note added: "A primitive low pass filter that is voltage controlled using a Vactrol.\nVery low cost device, but note that it draws a bit more current than CV\ninputs normally do. Running several in parallell probably requires a \nseparate splitter/mult."
- note added: "NOTE:\n- Filter caps and slew cap(s) can be chosen according to taste.\n- The slew caps C1 and C2 can be replaced with one bipolar, e.g. 470uF capacitor.\n- With both filters off it becomes more of a VCA, no filtering.\n- RV1 is way too big for this application, feel free to try a smaller value.\n- R3 is there because RV1 is too big (no effect on upper half of pot sweep).\n- R2 is there because o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"
- note removed: "NOTE:\n- Filter caps and slew cap(s) can be chosen according to taste.\n- The slew caps C1 and C2 can be replaced with one bipolar 470uF capacitor.\n- With both filters off it becomes more of a VCA, no filtering.\n- R3 is there basically because RV1 is way too big (no effect on upper half of pot sweep).\n- R2 is there because of a dead spot at the lower end of the sweep. Could use a resistor of 1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"
- moved on the sheet: C3, C4, R3, RV2
