File: supersimplesequencer/schematic/SSS1.kicad_pcb (KiCad board)
At the start: 2 copper layers, 61 parts, among them J1 RESET_IN, J2 CLK_IN, J3 STEP1_OUT, J4 CV1_OUT, J5 CV2_OUT, J6 GATE_OUT, J7 POWER, SW1 CV2_SCALE, U1 40106-pwr, U2 4017-pwr, U3 NE555, U4 LM324

Commit message: Update SSS-1 to beyond prototype
Adding features after using the stripboard prototype a bit, like e.g.:
- Searate output for all steps.
- Using 12V logic (will probably use the small connector for all PCBs).
- Switch for hold/run.
- Switch for step.
- Switch for reset.

The last three untested at this time.
Parts:
- removed D17, D18, D19: 1N4148, Diodes_THT:D_A-405_P7.62mm_Horizontal
- removed J5: CV2_OUT, Socket_Strips:Socket_Strip_Straight_1x03_Pitch2.54mm
- removed J6: GATE_OUT, Socket_Strips:Socket_Strip_Straight_1x03_Pitch2.54mm
- removed J7: POWER, Pin_Headers:Pin_Header_Straight_2x08_Pitch2.54mm
- added C10: 100nF, Capacitors_THT:C_Rect_L7.2mm_W3.5mm_P5.00mm_FKS2_FKP2_MKS2_MKP2, F.Cu at (344.6, 45.0)
- added C11: 100nF, Capacitors_THT:C_Rect_L7.2mm_W3.5mm_P5.00mm_FKS2_FKP2_MKS2_MKP2, F.Cu at (331.7, 66.5)
- added C12: 100nF, Capacitors_THT:C_Rect_L7.2mm_W3.5mm_P5.00mm_FKS2_FKP2_MKS2_MKP2, F.Cu at (342.2, 53.2)
- added C13: 100nF, Capacitors_THT:C_Rect_L7.2mm_W3.5mm_P5.00mm_FKS2_FKP2_MKS2_MKP2, F.Cu at (307.3, 90.5)
- added C14: 100nF, Capacitors_THT:C_Rect_L7.2mm_W3.5mm_P5.00mm_FKS2_FKP2_MKS2_MKP2, F.Cu at (323.3, 73.2)
- added C15: 100nF, Capacitors_THT:C_Rect_L7.2mm_W3.5mm_P5.00mm_FKS2_FKP2_MKS2_MKP2, F.Cu at (297.1, 98.7)
- added C16: 100nF, Capacitors_THT:C_Rect_L7.2mm_W3.5mm_P5.00mm_FKS2_FKP2_MKS2_MKP2, F.Cu at (323.3, 65.0)
- added C17: 100nF, Capacitors_THT:C_Rect_L7.2mm_W3.5mm_P5.00mm_FKS2_FKP2_MKS2_MKP2, F.Cu at (315.0, 77.7)
- added C18: 100nF, Capacitors_THT:C_Rect_L7.2mm_W3.5mm_P5.00mm_FKS2_FKP2_MKS2_MKP2, F.Cu at (286.9, 105.3)
- added C7: 10uF, Capacitors_THT:CP_Radial_D5.0mm_P2.00mm, F.Cu at (113.0, 139.7)
- added C8: 10uF, Capacitors_THT:CP_Radial_D5.0mm_P2.00mm, F.Cu at (114.3, 146.1)
- added C9: 100nF, Capacitors_THT:C_Rect_L7.2mm_W3.5mm_P5.00mm_FKS2_FKP2_MKS2_MKP2, F.Cu at (332.0, 58.3)
- added R16: 220k, Resistors_THT:R_Axial_DIN0207_L6.3mm_D2.5mm_P7.62mm_Horizontal, F.Cu at (304.4, 68.7)
- added R17: 100k, Resistors_THT:R_Axial_DIN0207_L6.3mm_D2.5mm_P7.62mm_Horizontal, F.Cu at (288.4, 83.1)
- added R18: 100, Resistors_THT:R_Axial_DIN0207_L6.3mm_D2.5mm_P7.62mm_Horizontal, F.Cu at (311.2, 62.1)
- added R19: 5.6k, Resistors_THT:R_Axial_DIN0207_L6.3mm_D2.5mm_P7.62mm_Horizontal, F.Cu at (334.0, 37.6)
- added R20: 2.7M, Resistors_THT:R_Axial_DIN0207_L6.3mm_D2.5mm_P7.62mm_Horizontal, F.Cu at (294.2, 76.4)
- added R21: 100k, Resistors_THT:R_Axial_DIN0207_L6.3mm_D2.5mm_P7.62mm_Horizontal, F.Cu at (266.1, 103.9)
- added R22: 100k, Resistors_THT:R_Axial_DIN0207_L6.3mm_D2.5mm_P7.62mm_Horizontal, F.Cu at (323.8, 44.2)
- added R23: 100k, Resistors_THT:R_Axial_DIN0207_L6.3mm_D2.5mm_P7.62mm_Horizontal, F.Cu at (255.6, 113.9)
- added R24: 100k, Resistors_THT:R_Axial_DIN0207_L6.3mm_D2.5mm_P7.62mm_Horizontal, F.Cu at (278.2, 91.4)
- added R25: 100k, Resistors_THT:R_Axial_DIN0207_L6.3mm_D2.5mm_P7.62mm_Horizontal, F.Cu at (311.2, 55.4)
- added R26: 100k, Resistors_THT:R_Axial_DIN0207_L6.3mm_D2.5mm_P7.62mm_Horizontal, F.Cu at (278.2, 84.8)
- added R27: 100k, Resistors_THT:R_Axial_DIN0207_L6.3mm_D2.5mm_P7.62mm_Horizontal, F.Cu at (294.2, 69.7)
- added R28: 100k, Resistors_THT:R_Axial_DIN0207_L6.3mm_D2.5mm_P7.62mm_Horizontal, F.Cu at (245.4, 117.2)
- added R29: 100k, Resistors_THT:R_Axial_DIN0207_L6.3mm_D2.5mm_P7.62mm_Horizontal, F.Cu at (255.9, 107.2)
- added R30: 100k, Resistors_THT:R_Axial_DIN0207_L6.3mm_D2.5mm_P7.62mm_Horizontal, F.Cu at (255.9, 100.6)
- added R31: 82k, Resistors_THT:R_Axial_DIN0207_L6.3mm_D2.5mm_P7.62mm_Horizontal, F.Cu at (331.6, 50.9)
- added R32: 82k, Resistors_THT:R_Axial_DIN0207_L6.3mm_D2.5mm_P7.62mm_Horizontal, F.Cu at (265.8, 117.2)
- added R33: 22k, Resistors_THT:R_Axial_DIN0207_L6.3mm_D2.5mm_P7.62mm_Horizontal, F.Cu at (298.6, 83.1)
- added R34: 100, Resistors_THT:R_Axial_DIN0207_L6.3mm_D2.5mm_P7.62mm_Horizontal, F.Cu at (276.3, 104.8)
- added R35: 100, Resistors_THT:R_Axial_DIN0207_L6.3mm_D2.5mm_P7.62mm_Horizontal, F.Cu at (344.2, 37.6)
- added R36: 100, Resistors_THT:R_Axial_DIN0207_L6.3mm_D2.5mm_P7.62mm_Horizontal, F.Cu at (334.0, 44.2)
- added R37: 100, Resistors_THT:R_Axial_DIN0207_L6.3mm_D2.5mm_P7.62mm_Horizontal, F.Cu at (304.4, 75.4)
- added R38: 100, Resistors_THT:R_Axial_DIN0207_L6.3mm_D2.5mm_P7.62mm_Horizontal, F.Cu at (321.4, 57.6)
- added R39: 100, Resistors_THT:R_Axial_DIN0207_L6.3mm_D2.5mm_P7.62mm_Horizontal, F.Cu at (288.4, 89.7)
- added R40: 100, Resistors_THT:R_Axial_DIN0207_L6.3mm_D2.5mm_P7.62mm_Horizontal, F.Cu at (276.3, 98.1)
- added R41: 100, Resistors_THT:R_Axial_DIN0207_L6.3mm_D2.5mm_P7.62mm_Horizontal, F.Cu at (266.1, 110.6)
- added R42: 100, Resistors_THT:R_Axial_DIN0207_L6.3mm_D2.5mm_P7.62mm_Horizontal, F.Cu at (321.4, 50.9)
- added RV10: B25k, Potentiometers:Potentiometer_Alps_RK09Y_Vertical, F.Cu at (168.9, 158.8)
- added RV11: 20k, Potentiometers:Potentiometer_Trimmer_Vishay_T73XX_Vertical, F.Cu at (311.7, 37.3)
- added RV12: 20k, Potentiometers:Potentiometer_Trimmer_Vishay_T73XX_Vertical, F.Cu at (250.4, 99.1)
- added RV13: 20k, Potentiometers:Potentiometer_Trimmer_Vishay_T73XX_Vertical, F.Cu at (305.5, 37.3)
- added SW2: STEP, Pin_Headers:Pin_Header_Straight_2x01_Pitch2.54mm, F.Cu at (148.6, 47.0)
- added SW3: HOLD_RUN, Pin_Headers:Pin_Header_Straight_1x03_Pitch2.54mm, F.Cu at (252.4, 87.6)
- added SW4: CV2_SCALE, Socket_Strips:Socket_Strip_Straight_1x03_Pitch2.54mm, F.Cu at (238.2, 101.7)
- added U5: TL074, Housings_DIP:DIP-14_W7.62mm_LongPads, F.Cu at (100.3, 31.8)
- added U6: TL074, Housings_DIP:DIP-14_W7.62mm_LongPads, F.Cu at (123.2, 120.7)
- added U7: TL074, Housings_DIP:DIP-14_W7.62mm_LongPads, F.Cu at (121.9, 97.8)
- C1: footprint Capacitors_THT:C_Rect_L9.0mm_W3.3mm_P7.50mm_MKT -> Capacitors_THT:C_Rect_L7.2mm_W3.5mm_P5.00mm_FKS2_FKP2_MKS2_MKP2
- C2: value 4.7uF -> 100nF; footprint Capacitors_THT:CP_Radial_D10.0mm_P5.00mm -> Capacitors_THT:C_Rect_L7.2mm_W3.5mm_P5.00mm_FKS2_FKP2_MKS2_MKP2
- C3: value 10uF -> 4.7uF; footprint Capacitors_THT:CP_Radial_D10.0mm_P5.00mm -> Capacitors_THT:CP_Radial_D5.0mm_P2.00mm
- C4: value CP -> 10uF; footprint Capacitors_THT:CP_Radial_D10.0mm_P5.00mm -> Capacitors_THT:CP_Radial_D5.0mm_P2.00mm
- C5, C6: value CP -> 100nF; footprint Capacitors_THT:CP_Radial_D10.0mm_P5.00mm -> Capacitors_THT:C_Rect_L7.2mm_W3.5mm_P5.00mm_FKS2_FKP2_MKS2_MKP2
- D11, D12, D13, D14, D15: value 1N4148 -> LED; footprint Diodes_THT:D_A-405_P7.62mm_Horizontal -> LEDs:LED_D3.0mm
- D3, D4: value LED -> 1N4148; footprint LEDs:LED_D3.0mm -> Diodes_THT:D_A-405_P7.62mm_Horizontal
- D6, D7: value LED -> 1N4001
- J3: value STEP1_OUT -> POWER; footprint Socket_Strips:Socket_Strip_Straight_1x03_Pitch2.54mm -> Pin_Headers:Pin_Header_Straight_2x05_Pitch2.54mm
- J4: value CV1_OUT -> OUTPUTS; footprint Socket_Strips:Socket_Strip_Straight_1x03_Pitch2.54mm -> Pin_Headers:Pin_Header_Straight_1x12_Pitch2.54mm
- R1, R2, R7, R8: value 100k -> 10k
- R10: value 100k -> 470
- R11: value 330 -> 12k
- R12: value 330 -> 220k
- R13: value 330 -> 100k
- R14: value 330 -> 100
- R15: value 5.6k -> 1k
- R3: value 2.2k -> 10k
- R4: value 12k -> 10k
- R5: value 470 -> 100k
- R9: value 100k -> 2.2k
- RV2: value B25k -> 100k; footprint Potentiometers:Potentiometer_Alps_RK09Y_Vertical -> Potentiometers:Potentiometer_Trimmer_Vishay_T73XX_Vertical
- SW1: value CV2_SCALE -> RESET; footprint Socket_Strips:Socket_Strip_Straight_1x03_Pitch2.54mm -> Pin_Headers:Pin_Header_Straight_2x01_Pitch2.54mm
- U4: value LM324 -> 4011; footprint Housings_DIP:DIP-14_W7.62mm_Socket_LongPads -> Housings_DIP:DIP-14_W7.62mm_LongPads
- moved SW1 239.9 mm to (348.7, 60.6)
- moved R11 234.1 mm to (308.7, 51.9)
- moved C5 217.1 mm to (299.0, 90.5)
- moved R14 208.9 mm to (311.2, 48.7)
- moved C6 198.5 mm to (276.7, 112.2)
- moved R2 188.5 mm to (319.2, 43.2)
- moved C4 188.0 mm to (245.1, 147.3)
- moved R13 180.6 mm to (301.0, 58.6)
- moved D1 172.1 mm to (282.7, 64.4)
- moved U4 166.7 mm to (147.3, 15.2)
- moved D11 162.6 mm to (350.3, 53.1)
- moved R1 159.6 mm to (270.0, 99.3)
- moved R7 159.1 mm to (257.8, 93.9)
- moved D6 150.7 mm to (342.6, 59.1)
- moved R10 149.2 mm to (267.0, 80.3)
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Connections:
- C3 pad 1: Net-(C2-Pad1) -> Net-(C3-Pad1)
- C4 pad 1: +5V -> Net-(C3-Pad1)
- C5 pad 1: +12V -> Net-(C5-Pad1)
- C6 pad 1: GND -> Net-(C6-Pad1)
- C6 pad 2: -12V -> GND
- D10 pad 2: STEP8 -> STEP3
- D11 pad 1: Net-(D11-Pad1) -> Net-(D10-Pad1)
- D11 pad 2: Net-(D11-Pad2) -> STEP4
- D12 pad 1: Net-(D11-Pad1) -> Net-(D10-Pad1)
- D12 pad 2: Net-(D12-Pad2) -> STEP5
- D13 pad 1: Net-(D11-Pad1) -> Net-(D10-Pad1)
- D13 pad 2: Net-(D13-Pad2) -> STEP6
- D14 pad 1: Net-(D11-Pad1) -> Net-(D10-Pad1)
- D14 pad 2: Net-(D14-Pad2) -> STEP7
- D15 pad 1: Net-(D11-Pad1) -> Net-(D10-Pad1)
- D15 pad 2: Net-(D15-Pad2) -> STEP8
- D16 pad 1: Net-(D11-Pad1) -> Net-(D16-Pad1)
- D16 pad 2: Net-(D16-Pad2) -> Net-(D10-Pad1)
- D3 pad 1: Net-(D10-Pad1) -> Net-(D3-Pad1)
- D3 pad 2: STEP1 -> Net-(D3-Pad2)
- D4 pad 1: Net-(D10-Pad1) -> Net-(D3-Pad1)
- D4 pad 2: STEP2 -> Net-(D4-Pad2)
- D5 pad 1: Net-(D10-Pad1) -> Net-(D5-Pad1)
- D5 pad 2: STEP3 -> Net-(D3-Pad1)
- D6 pad 1: Net-(D10-Pad1) -> +12V
- D6 pad 2: STEP4 -> GND
- D7 pad 1: Net-(D10-Pad1) -> GND
- D7 pad 2: STEP5 -> -12V
- D8 pad 2: STEP6 -> STEP1
- D9 pad 2: STEP7 -> STEP2
- J3 pad 1: Net-(J3-Pad1) -> -12V
- J3 pad 2: GND -> -12V
- J3 pad 3: Net-(J3-Pad3) -> GND
- J4 pad 2: GND -> Net-(J4-Pad2)
- R1 pad 1: Net-(D1-Pad1) -> +12V
- R1 pad 2: Net-(J2-Pad1) -> Net-(R1-Pad2)
- R10 pad 2: GND -> Net-(R10-Pad2)
- R11 pad 1: Net-(J5-Pad1) -> +12V
- R11 pad 2: Net-(R11-Pad2) -> Net-(J2-Pad3)
- R12 pad 1: Net-(J3-Pad1) -> GND
- R13 pad 1: Net-(J4-Pad1) -> Net-(R13-Pad1)
- R13 pad 2: Net-(R13-Pad2) -> Net-(R12-Pad2)
- R14 pad 1: Net-(J6-Pad1) -> CLK_OUT
- R14 pad 2: Net-(R14-Pad2) -> Net-(R13-Pad1)
- R15 pad 1: GND -> Net-(D5-Pad1)
- R15 pad 2: Net-(D19-Pad1) -> GND
- R2 pad 1: Net-(D2-Pad1) -> Net-(C1-Pad1)
- R2 pad 2: Net-(J1-Pad1) -> Net-(R1-Pad2)
- R3 pad 1: Net-(R3-Pad1) -> +12V
- R3 pad 2: Net-(C2-Pad1) -> Net-(R3-Pad2)
- R4 pad 1: +5V -> +12V
- R4 pad 2: Net-(J2-Pad3) -> Net-(R4-Pad2)
- R5 pad 1: Net-(R5-Pad1) -> Net-(D1-Pad1)
- R5 pad 2: Net-(R5-Pad2) -> Net-(J2-Pad1)
- R6 pad 1: Net-(R6-Pad1) -> Net-(D2-Pad1)
- R6 pad 2: GND -> Net-(J1-Pad1)
- R7 pad 1: Net-(R13-Pad2) -> Net-(C5-Pad1)
- R7 pad 2: Net-(R7-Pad2) -> Net-(R3-Pad2)
- R8 pad 1: Net-(R6-Pad1) -> Net-(C6-Pad1)
- R8 pad 2: GND -> Net-(R4-Pad2)
- R9 pad 1: Net-(R6-Pad1) -> Net-(R9-Pad1)
- R9 pad 2: GND -> Net-(C3-Pad1)
- RV1 pad 1: Net-(R5-Pad2) -> Net-(R10-Pad2)
- RV1 pad 2: Net-(R3-Pad1) -> Net-(R9-Pad1)
- RV1 pad 3: Net-(C2-Pad1) -> Net-(C3-Pad1)
- RV2 pad 1: STEP1 -> -12V
- RV2 pad 2: Net-(D11-Pad2) -> Net-(R20-Pad2)
- RV3 pad 1: STEP2 -> STEP1
- RV3 pad 2: Net-(D12-Pad2) -> Net-(R21-Pad2)
- RV4 pad 1: STEP3 -> STEP2
- RV4 pad 2: Net-(D13-Pad2) -> Net-(R22-Pad2)
- RV5 pad 1: STEP4 -> STEP3
- RV5 pad 2: Net-(D14-Pad2) -> Net-(R23-Pad2)
- RV6 pad 1: STEP5 -> STEP4
- RV6 pad 2: Net-(D15-Pad2) -> Net-(R24-Pad2)
- RV7 pad 1: STEP6 -> STEP5
- RV7 pad 2: Net-(D16-Pad2) -> Net-(R25-Pad2)
- RV8 pad 1: STEP7 -> STEP6
- RV9 pad 1: STEP8 -> STEP7
- SW1 pad 1: Net-(R10-Pad1) -> GND
- SW1 pad 2: Net-(R7-Pad2) -> Net-(R1-Pad2)
- U1 pad 11: Net-(D2-Pad1) -> Net-(C1-Pad1)
- U1 pad 14: +5V -> +12V
- U1 pad 3: Net-(U1-Pad2) -> Net-(C6-Pad1)
- U1 pad 4: CLK -> Net-(U1-Pad4)
- U1 pad 5: (no net) -> Net-(C5-Pad1)
- U1 pad 6: (no net) -> Net-(D3-Pad2)
- U1 pad 8: (no net) -> Net-(U1-Pad8)
- U1 pad 9: (no net) -> Net-(D2-Pad1)
- U2 pad 11: Net-(U2-Pad11) -> (no net)
- U2 pad 12: Net-(U2-Pad12) -> (no net)
- U2 pad 14: CLK -> Net-(D3-Pad1)
- U2 pad 15: Net-(U1-Pad12) -> Net-(U2-Pad15)
- U2 pad 16: +5V -> +12V
- U3 pad 2: Net-(C2-Pad1) -> Net-(C3-Pad1)
- U3 pad 3: Net-(R5-Pad1) -> Net-(R10-Pad1)
- U3 pad 4: +5V -> +12V
- U3 pad 5: Net-(C1-Pad1) -> Net-(C2-Pad1)
- U3 pad 6: Net-(C2-Pad1) -> Net-(C3-Pad1)
- U3 pad 8: +5V -> +12V
- U4 pad 1: Net-(R13-Pad2) -> Net-(U1-Pad2)
- U4 pad 10: CLK -> Net-(U4-Pad10)
- U4 pad 11: -12V -> Net-(D4-Pad2)
- U4 pad 12: STEP1 -> Net-(U4-Pad10)
- U4 pad 13: Net-(R12-Pad2) -> Net-(U4-Pad10)
- U4 pad 14: Net-(R12-Pad2) -> +12V
- U4 pad 2: Net-(R13-Pad2) -> Net-(U1-Pad2)
- U4 pad 3: Net-(D11-Pad1) -> Net-(U4-Pad3)
- U4 pad 4: +12V -> Net-(U2-Pad15)
- U4 pad 5: Net-(R7-Pad2) -> Net-(U1-Pad12)
- U4 pad 6: Net-(R11-Pad2) -> Net-(U1-Pad8)
- U4 pad 7: Net-(R11-Pad2) -> GND
- U4 pad 8: Net-(R14-Pad2) -> Net-(U1-Pad4)
- U4 pad 9: Net-(R14-Pad2) -> Net-(U4-Pad3)
