File: mini-lpg/kicad_files/minilpg.kicad_pcb (KiCad board)
At the start: 2 copper layers, 80 x 41.9 mm, 25 parts, among them J1 CV, J2 IN, J3 OUT, SW1 LP/BP, SW2 LPG/VCA, SW3 MINIDIST, U1 NSL-32

Commit message: Ringmod and minimod layout done
Routing:
- net GND: track 229.6 -> 164.9 mm
Other:
- board text added: "audio input"
- board text added: "audio output"
- board text added: "cutoff"
- board text added: "cv input"
- board text added: "dist"
- board text added: "low / band"
- board text added: "lpg / vca"
- board text added: "mini-lpg"
- board text added: "mini-lpg, rev A electronic sound machines, (c) 2018 uheriks@yahoo.ca"

Commit message: Final touches to ringmod/LPG PCB for rev A
Parts:
- moved J1 1.27 mm to (147.3, 64.8)
- moved J3 1.27 mm to (193.0, 64.8)
- moved J2 1.07 mm to (170.2, 64.8)
Routing:
- net GND: track 164.9 -> 166.7 mm
- net Net-(J1-Pad1): track 46.8 -> 47.9 mm
- net Net-(R3-Pad1): track 27.6 -> 28.6 mm
- net Net-(J3-Pad1): track 43.9 -> 44.9 mm
Other:
- board text added: "electronic sound machines"
- board text added: "mini-lpg, rev A electronic sound machines (c) 2018 Håkan Eriksson uheriks@yahoo.ca"
- board text removed: "mini-lpg, rev A electronic sound machines, (c) 2018 uheriks@yahoo.ca"
