File: ringmod/kicad_files/ringmod.kicad_pcb (KiCad board)
At the start: 2 copper layers, 71.1 x 41.9 mm, 13 parts, among them J1 CARRIER, J2 IN, J3 OUT

Commit message: Final touches to ringmod/LPG PCB for rev A
Parts:
- moved J1 1.27 mm to (136.5, 121.3)
- moved J2 1.27 mm to (159.4, 121.3)
- moved J3 1.27 mm to (182.2, 121.3)
Routing:
- net Net-(D2-Pad1): track 12.3 -> 22.2 mm
- net Net-(J3-Pad1): track 28.6 -> 31.8 mm
- net Net-(J2-Pad2): track 40.7 -> 43.5 mm
- net Net-(J2-Pad1): track 43.9 -> 46.4 mm
- net Net-(D1-Pad2): track 27.2 -> 28.9 mm
- net Net-(D3-Pad2): track 28.1 -> 29.4 mm
- net Net-(J3-Pad2): track 24.6 -> 25.6 mm
- net Net-(J1-Pad1): track 90.4 -> 91.4 mm
- net Net-(D1-Pad1): track 11.7 -> 11.2 mm
Other:
- board text added: "electronic sound machines"
- board text added: "mini-ringmod, rev A electronic sound machines (c) 2018, Håkan Eriksson uheriks@yahoo.ca"
- board text removed: "mini-ringmod, rev A electronic sound machines, (c) 2018 uheriks@yahoo.ca"
