File: slew_motion/kicad_files/slewmotion.sch (KiCad schematic (older format))
At the start: 115 parts

Commit message: Lots of changes, not sure what is what
Parts:
- C1, C2, C3, C4, C5, C6, C7, C8: renamed from C?; symbol C -> Device:C
- D1, D2, D3, D4, D5, D6, D7, D8, D9: renamed from D?; symbol 1N4148 -> Diode:1N4148
- J1, J2: renamed from J?; symbol Audio-Jack-2_Switch -> slewmotion-rescue:Audio-Jack-2_Switch
- J3, J4, J5, J6, J7, J8: renamed from J?; symbol Audio-Jack-2 -> slewmotion-rescue:Audio-Jack-2
- Q1, Q2, Q3, Q4: renamed from Q?; symbol BC337 -> slewmotion-rescue:BC337
- R1, R10, R11, R12, R13, R14, R15, R16, R17, R18, R19, R2, R20, R21, R22, R23, R24, R25, R26, R27, R28, R29, R3, R30, R31, R32, R33, R34, R35, R36, R37, R38, R39, R4, R40, R41, R42, R43, R44, R45, R46, R47, R48, R49, R5, R50, R51, R52, R53, R54, R55, R6, R7, R8, R9: renamed from R?; symbol R -> Device:R
- RV1, RV2, RV3, RV4, RV5, RV6, RV7, RV8: renamed from RV?; symbol POT -> slewmotion-rescue:POT
- SW1, SW4: renamed from SW?; symbol SW_Push -> slewmotion-rescue:SW_Push
- SW2, SW3, SW5, SW6: renamed from SW?; symbol SW_SPST -> slewmotion-rescue:SW_SPST
- U1, U4: renamed from U?; symbol 40106 -> slewmotion-rescue:40106
- U2, U3: renamed from U?; symbol TL074 -> slewmotion-rescue:TL074
Connections:
- net GND: now also U2.10 (+), U2.12 (+), U2.5 (+), U3.5 (+); no longer U2.3 (+), U2.3 (+), U2.3 (+), U3.3 (+)
- net at R26.1, R38.2: now also U2.8, U3.9 (-); no longer U2.1, U3.2 (-)
- net at R24.2, R26.2: now also U2.9 (-); no longer U2.2 (-)
- net at C7.2, R46.2: now also U1.13 (In); no longer U1.1 (In)
- net at RV8.2, RV8.3: now also U1.12 (Out), U4.3 (In); no longer U1.2 (Out), U4.1 (In)
- net at C7.1, R15.2, R48.2: now also U1.8 (Out); no longer U1.2 (Out)
- net at R35.1, R37.2: now also U3.7; no longer U3.1
- net at R29.2, R35.2: now also U3.6 (-); no longer U3.2 (-)
- net at R30.1, R32.1, R39.2: now also U3.10 (+); no longer U3.3 (+)
- net at C6.1, RV8.1: now also U1.5 (In); no longer U1.1 (In)
- net at D5.2 (A): now also U1.6 (Out); no longer U1.2 (Out)
- net at R23.1, RV5.1, RV6.1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: now also U2.7; no longer U2.1
- net at R19.2, R20.2, R21.2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: now also U2.6 (-); no longer U2.2 (-)
- net at R27.1, R40.2: now also U2.14, U3.13 (-); no longer U2.1, U3.2 (-)
- net at R25.2, R27.2: now also U2.13 (-); no longer U2.2 (-)
- net at RV7.2, RV7.3, U4.2 (Out): now also U4.5 (In); no longer U4.1 (In)
- net at C8.1, R2.1, R49.2: now also U1.10 (Out); no longer U1.2 (Out)
- net at R31.1, R33.1, R41.2: now also U3.12 (+); no longer U3.3 (+)
- net at C5.1, RV7.1: now also U1.3 (In); no longer U1.1 (In)
- net at SW6.2 (B): now also U1.4 (Out); no longer U1.2 (Out)
- net at R53.2: now also U4.6 (Out); no longer U4.2 (Out)
- net at R52.2: now also U4.4 (Out); no longer U4.2 (Out)
- new net: R39.1, U1.9 (In), U3.8
- new net: R41.1, U1.11 (In), U3.14
Other:
- note added: "NOTE: Bipolar electrolyte?\n"
