File: triggerhappy/kicad_files/triggerhappy.kicad_pcb (KiCad board)
At the start: 2 copper layers, 49.9 x 99.8 mm, 70 parts, among them J1 EUROPOWER, J2 GATE_IN, J3 TRIG_1, J4 TRIG_2, J5 TRIG_3, J6 TRIG_4, J7 TRIG_5, J8 TRIG_MIX, U1 40106-pwr, U2 40106-pwr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

Commit message: triggerhappy: Add text
Other:
- board text added: "all aboard"
Changed lines of the file:
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@@
   (general
     (thickness 1.6)
-    (drawings 9)
+    (drawings 10)
     (tracks 305)
     (zones 0)
@@
       (net 21 "Net-(D7-Pad1)"))
   )
+  (gr_text "all\naboard" (at 211.074 100.203 45) (layer F.SilkS)
+    (effects (font (size 1 1) (thickness 0.1)))
+  )
   (gr_text "Jacks: PJ301BM (from Thonk)\nPots: Song Huei 9mm vertical pot (Thonk)" (at 196.85 172.974) (layer Cmts.User)

Commit message: minidrum: Move switches apart a bit
Experiments with PCB layout on paper indicated that the
space between switches was too tight. Maybe still, but better.

Also cleaning up other PCBs a bit.
Other:
- board text added: "boing boom"
- board text added: "triggerhappy"
- board text added: "triggerhappy, rev A electronic sound machines (c) 2019, Håkan Eriksson uheriks@yahoo.ca"
- board text added: "tschak"
- board text removed: "all aboard"
- board text removed: "trigtrain"
- board text removed: "trigtrain, rev A electronic sound machines (c) 2019, Håkan Eriksson uheriks@yahoo.ca"
Changed lines of the file:
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@@
   (general
     (thickness 1.6)
-    (drawings 10)
+    (drawings 11)
     (tracks 305)
     (zones 0)
@@
       (net 21 "Net-(D7-Pad1)"))
   )
-  (gr_text "all\naboard" (at 211.074 100.203 45) (layer F.SilkS)
+  (gr_text tschak (at 226.822 95.631 90) (layer F.SilkS)
+    (effects (font (size 1 1) (thickness 0.1)))
+  )
+  (gr_text "boing\nboom" (at 211.074 100.203 45) (layer F.SilkS)
     (effects (font (size 1 1) (thickness 0.1)))
   )
@@
     (effects (font (size 1.5 1.5) (thickness 0.3)))
   )
-  (gr_text trigtrain (at 200.66 189.484) (layer Cmts.User)
+  (gr_text triggerhappy (at 200.66 189.484) (layer Cmts.User)
     (effects (font (size 1.5 1.5) (thickness 0.3)))
   )
-  (gr_text "trigtrain, rev A\nelectronic sound machines\n(c) 2019, Håkan Eriksson\n\nuheriks@yahoo.ca" (at 206.883 116.84) (layer F.SilkS)
+  (gr_text "triggerhappy, rev A\nelectronic sound machines\n(c) 2019, Håkan Eriksson\n\nuheriks@yahoo.ca" (at 206.883 116.84) (layer F.SilkS)
     (effects (font (size 1 1) (thickness 0.2)))
   )
