File: triggerhappy/kicad_files/triggerhappy.sch (KiCad schematic (older format))
At the start: 69 parts, among them J1 EUROPOWER, J2 GATE_IN, J3 TRIG_1, J4 TRIG_2, J5 TRIG_3, J6 TRIG_4, J7 TRIG_5, J8 TRIG_MIX, U1 40106-pwr, U2 40106-pwr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

Commit message: Unknown changes in triggerhappy (not sure if in built PCB)
The changes were made on May 27 2019. Could probably figure out if it went into the PCB or not
Parts:
- added C?: 10uF, symbol Device:C
- added C? (x2): 100n, Capacitor_THT:C_Rect_L7.2mm_W2.5mm_P5.00mm_FKS2_FKP2_MKS2_MKP2, symbol Device:C
- added D? (x2): D, symbol Device:D
- added R?: 100k, symbol Device:R
- added R?: 10k, symbol Device:R
- added R?: 330k, MusicThingModular:7MM_RESISTOR, symbol Device:R
- added SW?: START, symbol Switch:SW_Push
- added SW?: LOOP, symbol Switch:SW_SPST
- added unit 3 of U1
- added unit 4 of U1
- C3: value 100n -> 470n
- R10, R11, R3, R8, R9: value 1k -> 1.5k
Connections:
- wire segments 241 -> 273
Other:
- note added: "These are not in rev A PCB, but they can be hacked in.\nFor manual start and loop respectively.\nNOTE: I think that letting gate in go directly to a Schmitt inverter\n(and build from that) could have made it possible to connect the \nloop signal with a patch cable. Will try that in the next build,\nthis is OK for now."
- note removed: "NOTE: It might to be possible to connect all the monstables’ diodes\nand connect them to the very first inverter. I chose completely \nseparate channels early, when it looked like the 555s input might \naffect other parts, but with the diode it should be ”isolated”. \nDon’t feel like testing that right now, having just finished the PCB\nand all, but for a potential rev B, perhaps?"
- note removed: "REMEMBER TO TEST THIS: \nShort delays on all, creating almost a drum sound, and run it through \nan LPG that is triggered by the same gate (with cap in series for \ndecay)."
- note removed: "WHEN BUILDING #1, don’t connect the diodes cathode side at first; \ntry hooking it up to pin 2 of the first inverter (to determine whether I \ncan skip four inverters => one entire chip can go."
