File: metallic_beat/kicad_files/metallic_beat.sch (KiCad schematic (older format))
At the start: 43 parts, among them J1 GATE_IN, J2 AUDIO_OUT, J3 POWER, Q1 BC337, Q2 BC547, Q3 BC547, U1 74HCT04, U2 74HCT04-pwr

Commit message: Add schematic PDF and readme for Metallic Beat
Other:
- note added: "NOTE:\nR12/C4 are there to shape the input gate into a trigger\nenvelope (since it's not a real CR-78, I have no control\nover the trig pulse). It's not ideal though, and could be\nreplaced with something smarter (maybe a monostable\nmultivibrator up front?)."
- note added: "NOTE:\nThere's one more transistor stage after Q3, \nfor amplification, will add later."
- note removed: "R12/C4 are there to shape the input gate into a trigger\nenvelope (since it's not a real CR-78, I have no control\nover the trig pulse). It's not ideal though, and could be\nreplaced with something smarter."
Changed lines of the file:
@@
 Connection ~ 6700 5000
 Connection ~ 3700 4500
-Text Notes 2000 7100 0    60   ~ 0
-R12/C4 are there to shape the input gate into a trigger\nenvelope (since it's not a real CR-78, I have no control\nover the trig pulse). It's not ideal though, and could be\nreplaced with something smarter.
+Text Notes 2000 7200 0    60   ~ 0
+NOTE:\nR12/C4 are there to shape the input gate into a trigger\nenvelope (since it's not a real CR-78, I have no control\nover the trig pulse). It's not ideal though, and could be\nreplaced with something smarter (maybe a monostable\nmultivibrator up front?).
 Text Notes 8150 7650 0    60   ~ 0
 March 21, 2018\n
@@
 Connection ~ 10400 1150
 Connection ~ 10400 1250
+Text Notes 7850 5300 0    60   ~ 0
+NOTE:\nThere's one more transistor stage after Q3, \nfor amplification, will add later.
 $EndSCHEMATC

Commit message: Lots of changes, not sure what is what
Parts:
- removed RV1: POT, symbol POT
- removed U1: 74HCT04, symbol 74HCT04-pwr
- removed U2: 74HCT04-pwr, symbol 74HCT04-pwr
- added C?: 100pF, symbol Device:C
- added C?: 4.7uF, symbol Device:CP
- added C? (x2): 100uF, symbol Device:CP
- added C? (x2): 100nF, symbol Device:C
- added JP?: IC_VCC_SEL, symbol Jumper:Jumper_3_Bridged12
- added Q?: BC337, Package_TO_SOT_THT:TO-92_Inline, symbol Transistor_BJT:BC337
- added R?: 120k, symbol Device:R
- added R?: 47k, symbol Device:R
- added R?: 470k, symbol Device:R
- added U? (x7): 4069, symbol 4xxx:4069
- C1, C2, C3, C4, C5, C6, C7: symbol C -> Device:C
- C8: value C -> 68nF; symbol C -> Device:C
- D1, D2: symbol D -> Device:D
- J1, J2: symbol Audio-Jack-2 -> metallic_beat-rescue:Audio-Jack-2
- J3: symbol Conn_02x08_Odd_Even -> metallic_beat-rescue:Conn_02x08_Odd_Even
- L1: symbol L -> Device:L
- Q1: symbol BC337 -> metallic_beat-rescue:BC337
- Q2, Q3: symbol BC547 -> metallic_beat-rescue:BC547
- R1, R10, R11, R12, R13, R14, R15, R16, R17, R18, R19, R2, R20, R21, R22, R23, R3, R4, R8, R9: symbol R -> Device:R
- R5, R6, R7: symbol RTRIM -> Device:RTRIM
Connections:
- net labels removed: -12V
- wire segments 99 -> 174
- no-connect marks 4 -> 6
Other:
- note added: "It ought to be possible to hack in pots for \nR16-R18 to be able to mix the waveforms.\nFor the overall valume it should be OK to adjust \nR19 (e.g. if driving the circuit with 12V results in\na too loud output)."
- note added: "NOTE:\nThe transistor after Q3 is only guessed, check built board?"
- note added: "Prototype warnings:\n——————————————\nThe IC is changed from my original prototype, as is\nthe IC voltage. Before hooking in the oscillator output \nto the transistor stages, add a volume pot in between.\nIf stuff doesn’t work, try running on 5V (and possibly \nswitch to the tested 74HCT04 – also listen for sound\nchanges).\n\nThe pulse shaping R12/C4 are probably not the best\nsolution. I chose t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"
- note added: "The chip in the original circuit runs on 5V, but if 5V is not \navailable it should be possible to run it on 12V.\nHave not tested, but should result in much higher levels,\nwhich should be solvable by lowering R19, perhaps?\nNot sure if it affects the frequencies.\n\nAlso, the original chip was MC14069. I have built one\nimplementation with a 74HCT04, and this (untested\nprototype) uses CD4069, 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"
- note removed: "NOTE:\nR12/C4 are there to shape the input gate into a trigger\nenvelope (since it's not a real CR-78, I have no control\nover the trig pulse). It's not ideal though, and could be\nreplaced with something smarter (maybe a monostable\nmultivibrator up front?)."
- note removed: "NOTE:\nThere's one more transistor stage after Q3, \nfor amplification, will add later."
- moved on the sheet: Q1

Commit message: Add trig capacitor jumper on Metallic Beat
Parts:
- added JP1: OPT_CAP, symbol Device:Jumper_NC_Small
- gave numbers to parts that had none: 12
Connections:
- wire segments 174 -> 175
Changed lines of the file:
@@
 	5100 6100 5100 5650
 Wire Wire Line
-	2000 6100 2700 6100
+	1900 6100 2700 6100
 Connection ~ 4600 6100
 Wire Wire Line
@@
 L metallic_beat-rescue:Audio-Jack-2 J1
 U 1 1 5AB07F43
-P 1800 5600
-F 0 "J1" H 1775 5675 50  0000 C CNN
-F 1 "GATE_IN" H 1775 5425 50  0000 C CNN
-F 2 "" H 2050 5600 50  0001 C CNN
-F 3 "" H 2050 5600 50  0001 C CNN
-	1    1800 5600
-	1    0    0    -1
-$EndComp
-Wire Wire Line
-	2000 5700 2000 6100
+P 1700 5600
+F 0 "J1" H 1675 5675 50  0000 C CNN
+F 1 "GATE_IN" H 1675 5425 50  0000 C CNN
+F 2 "" H 1950 5600 50  0001 C CNN
+F 3 "" H 1950 5600 50  0001 C CNN
+	1    1700 5600
+	1    0    0    -1
+$EndComp
+Wire Wire Line
+	1900 5700 1900 6100
 Wire Wire Line
 	2700 6100 2700 6000
@@
 	2700 5700 2700 5600
 Connection ~ 2700 5600
-Wire Wire Line
-	2300 5600 2000 5600
 Wire Wire Line
 	6700 4300 6700 4400
@@
 	9450 1400 9950 1400
 $Comp
-L Transistor_BJT:BC337 Q?
+L Transistor_BJT:BC337 Q4
 U 1 1 5BDB5BE1
 P 7700 5300
-F 0 "Q?" H 7891 5346 50  0000 L CNN
+F 0 "Q4" H 7891 5346 50  0000 L CNN
 F 1 "BC337" H 7891 5255 50  0000 L CNN
 F 2 "Package_TO_SOT_THT:TO-92_Inline" H 7900 5225 50  0001 L CIN
@@
 	6500 6100 7400 6100
 $Comp
-L Device:R R?
+L Device:R R24
 U 1 1 5BDBB394
 P 7400 5650
-F 0 "R?" H 7470 5696 50  0000 L CNN
+F 0 "R24" H 7470 5696 50  0000 L CNN
 F 1 "120k" H 7470 5605 50  0000 L CNN
 F 2 "" V 7330 5650 50  0001 C CNN
@@
 $EndComp
 $Comp
-L Device:R R?
+L Device:R R26
 U 1 1 5BDBB432
 P 7800 4550
-F 0 "R?" H 7870 4596 50  0000 L CNN
+F 0 "R26" H 7870 4596 50  0000 L CNN
 F 1 "47k" H 7870 4505 50  0000 L CNN
 F 2 "" V 7730 4550 50  0001 C CNN
@@
 Connection ~ 6700 4300
 $Comp
-L Device:R R?
+L Device:R R25
 U 1 1 5BDE303F
 P 7600 4800
-F 0 "R?" V 7393 4800 50  0000 C CNN
+F 0 "R25" V 7393 4800 50  0000 C CNN
 F 1 "470k" V 7484 4800 50  0000 C CNN
 F 2 "" V 7530 4800 50  0001 C CNN
@@
 $EndComp
 $Comp
-L Device:C C?
+L Device:C C11
 U 1 1 5BDED7C4
 P 7600 5000
-F 0 "C?" H 7625 5100 50  0000 L CNN
+F 0 "C11" H 7625 5100 50  0000 L CNN
 F 1 "100pF" H 7625 4900 50  0000 L CNN
 F 2 "" H 7638 4850 50  0001 C CNN
@@
 	7400 6100 7800 6100
 $Comp
-L Device:CP C?
+L Device:CP C12
 U 1 1 5BE08F76
 P 8250 5000
-F 0 "C?" V 8505 5000 50  0000 C CNN
+F 0 "C12" V 8505 5000 50  0000 C CNN
 F 1 "4.7uF" V 8414 5000 50  0000 C CNN
 F 2 "" H 8288 4850 50  0001 C CNN
@@
 The chip in the original circuit runs on 5V, but if 5V is not \navailable it should be possible to run it on 12V.\nHave not tested, but should result in much higher levels,\nwhich should be solvable by lowering R19, perhaps?\nNot sure if it affects the frequencies.\n\nAlso, the original chip was MC14069. I have built one\nimplementation with a 74HCT04, and this (untested\nprototype) uses CD4069, to be able to run it on 12V\n(which also is untested, and possibly pointless).
 $Comp
-L Jumper:Jumper_3_Bridged12 JP?
+L Jumper:Jumper_3_Bridged12 JP2
 U 1 1 5C490801
 P 8900 1150
-F 0 "JP?" H 8900 1262 50  0000 C CNN
+F 0 "JP2" H 8900 1262 50  0000 C CNN
 F 1 "IC_VCC_SEL" H 8900 1353 50  0000 C CNN
 F 2 "" H 8900 1150 50  0001 C CNN
@@
 	8650 1150 8650 900
 $Comp
-L Device:CP C?
+L Device:CP C13
 U 1 1 5C4BB612
 P 10350 1600
-F 0 "C?" H 10468 1646 50  0000 L CNN
+F 0 "C13" H 10468 1646 50  0000 L CNN
 F 1 "100uF" H 10468 1555 50  0000 L CNN
 F 2 "" H 10388 1450 50  0001 C CNN
@@
 $EndComp
 $Comp
-L Device:CP C?
+L Device:CP C10
 U 1 1 5C4ECA75
 P 7500 1250
-F 0 "C?" H 7618 1296 50  0000 L CNN
+F 0 "C10" H 7618 1296 50  0000 L CNN
 F 1 "100uF" H 7618 1205 50  0000 L CNN
 F 2 "" H 7538 1100 50  0001 C CNN
@@
 	10350 1750 10350 1800
 $Comp
-L Device:C C?
+L Device:C C14
 U 1 1 5C52718B
 P 10800 1600
-F 0 "C?" H 10915 1646 50  0000 L CNN
+F 0 "C14" H 10915 1646 50  0000 L CNN
 F 1 "100nF" H 10915 1555 50  0000 L CNN
 F 2 "" H 10838 1450 50  0001 C CNN
@@
 $EndComp
 $Comp
-L Device:C C?
+L Device:C C9
 U 1 1 5C5272EB
 P 7050 1250
-F 0 "C?" H 7165 1296 50  0000 L CNN
+F 0 "C9" H 7165 1296 50  0000 L CNN
 F 1 "100nF" H 7165 1205 50  0000 L CNN
 F 2 "" H 7088 1100 50  0001 C CNN
@@
 	9950 1700 10100 1700
 $Comp
-L 4xxx:4069 U?
+L 4xxx:4069 U1
 U 1 1 5C5C6DBC
 P 3150 1300
-F 0 "U?" H 3200 1150 50  0000 C CNN
+F 0 "U1" H 3200 1150 50  0000 C CNN
 F 1 "4069" H 3200 1450 50  0000 C CNN
 F 2 "" H 3150 1300 50  0001 C CNN
@@
 $EndComp
 $Comp
-L 4xxx:4069 U?
+L 4xxx:4069 U1
 U 2 1 5C5CF211
 P 4250 1300
-F 0 "U?" H 4300 1150 50  0000 C CNN
+F 0 "U1" H 4300 1150 50  0000 C CNN
 F 1 "4069" H 4300 1450 50  0000 C CNN
 F 2 "" H 4250 1300 50  0001 C CNN
@@
 $EndComp
 $Comp
-L 4xxx:4069 U?
+L 4xxx:4069 U1
 U 3 1 5C5CF2A0
 P 3150 2300
-F 0 "U?" H 3200 2150 50  0000 C CNN
+F 0 "U1" H 3200 2150 50  0000 C CNN
 F 1 "4069" H 3200 2450 50  0000 C CNN
 F 2 "" H 3150 2300 50  0001 C CNN
@@
 $EndComp
 $Comp
-L 4xxx:4069 U?
+L 4xxx:4069 U1
 U 4 1 5C5CF331
 P 4250 2300
-F 0 "U?" H 4300 2150 50  0000 C CNN
+F 0 "U1" H 4300 2150 50  0000 C CNN
 F 1 "4069" H 4300 2450 50  0000 C CNN
 F 2 "" H 4250 2300 50  0001 C CNN
@@
 $EndComp
 $Comp
-L 4xxx:4069 U?
+L 4xxx:4069 U1
 U 6 1 5C5CF3BC
 P 4250 3300
-F 0 "U?" H 4300 3150 50  0000 C CNN
+F 0 "U1" H 4300 3150 50  0000 C CNN
 F 1 "4069" H 4300 3450 50  0000 C CNN
 F 2 "" H 4250 3300 50  0001 C CNN
@@
 $EndComp
 $Comp
-L 4xxx:4069 U?
+L 4xxx:4069 U1
 U 5 1 5C5CF459
 P 3150 3300
-F 0 "U?" H 3200 3150 50  0000 C CNN
+F 0 "U1" H 3200 3150 50  0000 C CNN
 F 1 "4069" H 3200 3450 50  0000 C CNN
 F 2 "" H 3150 3300 50  0001 C CNN
@@
 $EndComp
 $Comp
-L 4xxx:4069 U?
+L 4xxx:4069 U1
 U 7 1 5C5CF74F
 P 8100 1350
-F 0 "U?" H 8250 1000 50  0000 C CNN
+F 0 "U1" H 8250 1000 50  0000 C CNN
 F 1 "4069" H 8250 1700 50  0000 C CNN
 F 2 "" H 8100 1350 50  0001 C CNN
@@
 	4550 3300 4800 3300
 Text Notes 550  7700 0    59   ~ 0
-Prototype warnings:\n——————————————\nThe IC is changed from my original prototype, as is\nthe IC voltage. Before hooking in the oscillator output \nto the transistor stages, add a volume pot in between.\nIf stuff doesn’t work, try running on 5V (and possibly \nswitch to the tested 74HCT04 – also listen for sound\nchanges).\n\nThe pulse shaping R12/C4 are probably not the best\nsolution. I chose to keep them in since I know they work\n(and I was to lazy to test new solutions). A capacitor in \nseries with the input should work fine, hence the jumper\nthere.\nIn the actual CR-78, the incoming pulse was obviously \ndesigned to have a certain length (and amplitude).
+Prototype warnings:\n——————————————\nThe IC is changed from my original prototype, as is\nthe IC voltage. Before hooking in the oscillator output \nto the transistor stages, add a volume pot in between.\nIf stuff doesn’t work, try running on 5V (and possibly \nswitch to the tested 74HCT04 – also listen for sound\nchanges).\n\nThe pulse shaping R12/C4 are probably not the best\nsolution. I chose to keep them in since I know they work\n(and I was to lazy to test new solutions). A capacitor in \nseries with the input should work fine, hence the jumper\nJ1 there (test that with no R12 and jumper over C4).\nIn the actual CR-78, the incoming pulse was obviously \ndesigned to have a certain length (and amplitude).
+$Comp
+L Device:Jumper_NC_Small JP1
+U 1 1 5C4DC16E
+P 2100 5600
+F 0 "JP1" H 2100 5812 50  0000 C CNN
+F 1 "OPT_CAP" H 2100 5721 50  0000 C CNN
+F 2 "" H 2100 5600 50  0001 C CNN
+F 3 "~" H 2100 5600 50  0001 C CNN
+	1    2100 5600
+	1    0    0    -1
+$EndComp
+Wire Wire Line
+	1900 5600 2000 5600
+Wire Wire Line
+	2200 5600 2300 5600
 $EndSCHEMATC

Commit message: Add test points and 5V filter resistor
Parts:
- added R?: 47, symbol Device:R
- added TP?: OSC_OUT, symbol Connector:TestPoint
- added TP?: OSC1_OUT, symbol Connector:TestPoint
- added TP?: OSC2_OUT, symbol Connector:TestPoint
- added TP?: OSC3_OUT, symbol Connector:TestPoint
Connections:
- wire segments 175 -> 180

Commit message: metallic beat: Finish PCB layout and routing
Parts:
- removed R5, R6, R7: 20k, symbol Device:RTRIM
- added D3: LOW POWER LED, LED_THT:LED_D3.0mm_FlatTop, symbol Device:LED
- added D4, D5: 1N4001, Diode_THT:D_DO-41_SOD81_P7.62mm_Horizontal, symbol Device:D
- added R28: 4.7k, Resistor_THT:R_Axial_DIN0207_L6.3mm_D2.5mm_P7.62mm_Horizontal, symbol Device:R
- added RV1, RV2, RV3: 20k, Potentiometer_THT:Potentiometer_Bourns_3386X_Horizontal, symbol Device:R_POT_TRIM
- added TP1: CAP1, TestPoint:TestPoint_THTPad_2.0x2.0mm_Drill1.0mm, symbol Connector:TestPoint
- added TP2: CAP2, TestPoint:TestPoint_THTPad_2.0x2.0mm_Drill1.0mm, symbol Connector:TestPoint
- added TP3: CAP3, TestPoint:TestPoint_THTPad_2.0x2.0mm_Drill1.0mm, symbol Connector:TestPoint
- C1, C11, C14, C2, C3, C4, C5, C6, C7, C8, C9: footprint (none) -> Capacitor_THT:C_Rect_L7.2mm_W2.5mm_P5.00mm_FKS2_FKP2_MKS2_MKP2
- C10, C13: value 100uF -> 10uF; footprint (none) -> Capacitor_THT:CP_Radial_D5.0mm_P2.00mm
- C12: footprint (none) -> Capacitor_THT:CP_Radial_D5.0mm_P2.00mm
- D1, D2: footprint (none) -> Diode_THT:D_DO-35_SOD27_P7.62mm_Horizontal
- J1, J2: footprint (none) -> kicadlib:Switchcraft_35RAPC2AV_3_5_mm_jack_no_switch
- J3: footprint (none) -> Connector_PinHeader_2.54mm:PinHeader_2x08_P2.54mm_Vertical
- JP1: footprint (none) -> Connector_PinHeader_2.54mm:PinHeader_1x02_P2.54mm_Vertical
- JP2: footprint (none) -> Connector_PinHeader_2.54mm:PinHeader_1x03_P2.54mm_Vertical
- L1: footprint (none) -> Inductor_THT:L_Radial_D12.0mm_P5.00mm_Fastron_11P
- Q1, Q2, Q3: footprint TO_SOT_Packages_THT:TO-92_Molded_Narrow -> Package_TO_SOT_THT:TO-92L
- Q4: footprint Package_TO_SOT_THT:TO-92_Inline -> Package_TO_SOT_THT:TO-92L
- R1, R10, R11, R12, R13, R14, R15, R16, R17, R18, R19, R2, R20, R21, R22, R23, R24, R25, R26, R3, R4, R8, R9: footprint (none) -> Resistor_THT:R_Axial_DIN0207_L6.3mm_D2.5mm_P7.62mm_Horizontal
- R27: renamed from R?; footprint (none) -> Resistor_THT:R_Axial_DIN0207_L6.3mm_D2.5mm_P7.62mm_Horizontal
- TP4: renamed from TP?; value OSC1_OUT -> OSC1; footprint (none) -> TestPoint:TestPoint_THTPad_2.0x2.0mm_Drill1.0mm
- TP5: renamed from TP?; value OSC2_OUT -> OSC2; footprint (none) -> TestPoint:TestPoint_THTPad_2.0x2.0mm_Drill1.0mm
- TP6: renamed from TP?; value OSC3_OUT -> OSC3; footprint (none) -> TestPoint:TestPoint_THTPad_2.0x2.0mm_Drill1.0mm
- TP7: renamed from TP?; footprint (none) -> TestPoint:TestPoint_THTPad_2.0x2.0mm_Drill1.0mm
- U1: footprint (none) -> Package_DIP:DIP-14_W7.62mm
Connections:
- wire segments 180 -> 210
Other:
- note added: "NOTE: It should be possible to change the oscillators’ frequency by \nadding a capacitor in parallell between the two test points in each sub-\ncircuit. The same value should (?) give half the frequency."
- note added: "NOTE: The LED might take too much of the gate\nsignal, test before committing to it!"
- note added: "Prototype warnings, untested stuff:\n——————————————————\nThe chip in the original circuit runs on 5V, but if 5V is not \navailable it should be possible to run it on 12V. It should\nresult in much higher levels, which should be solvable by\nlowering R19? Not sure if it affects the frequencies.\n\nAlso, the original chip was MC14069. I have built one\nimplementation with a 74HCT04, and this (untes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"
- note removed: "Prototype warnings:\n——————————————\nThe IC is changed from my original prototype, as is\nthe IC voltage. Before hooking in the oscillator output \nto the transistor stages, add a volume pot in between.\nIf stuff doesn’t work, try running on 5V (and possibly \nswitch to the tested 74HCT04 – also listen for sound\nchanges).\n\nThe pulse shaping R12/C4 are probably not the best\nsolution. I chose t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"
- note removed: "The chip in the original circuit runs on 5V, but if 5V is not \navailable it should be possible to run it on 12V.\nHave not tested, but should result in much higher levels,\nwhich should be solvable by lowering R19, perhaps?\nNot sure if it affects the frequencies.\n\nAlso, the original chip was MC14069. I have built one\nimplementation with a 74HCT04, and this (untested\nprototype) uses CD4069, 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"
- moved on the sheet: Q4

Commit message: metallic beat: Add jumper for VCA
Mainly for test and experimentation purposes, having a jumper in
the oscillator signal's path to the VCA/filter thing could be nice
to make it possible to run other things through there.

NOTE: When building,one will have to add a capacitor on the jack!
I figured the existing one would be too small to use as a
decoupling capacitor.
Parts:
- added JP3: VCA_IN, Connector_PinHeader_2.54mm:PinHeader_1x02_P2.54mm_Vertical, symbol Device:Jumper_NC_Small
Connections:
- wire segments 210 -> 211
Changed lines of the file:
@@
 L Device:C C6
 U 1 1 5AB052BF
-P 5600 3650
-F 0 "C6" H 5625 3750 50  0000 L CNN
-F 1 "15 nF" H 5300 3750 50  0000 L CNN
-F 2 "Capacitor_THT:C_Rect_L7.2mm_W2.5mm_P5.00mm_FKS2_FKP2_MKS2_MKP2" H 5638 3500 50  0001 C CNN
-F 3 "" H 5600 3650 50  0001 C CNN
-	1    5600 3650
+P 5600 3600
+F 0 "C6" H 5625 3700 50  0000 L CNN
+F 1 "15 nF" H 5350 3700 50  0000 L CNN
+F 2 "Capacitor_THT:C_Rect_L7.2mm_W2.5mm_P5.00mm_FKS2_FKP2_MKS2_MKP2" H 5638 3450 50  0001 C CNN
+F 3 "" H 5600 3600 50  0001 C CNN
+	1    5600 3600
 	-1   0    0    1
 $EndComp
@@
 $EndComp
 Wire Wire Line
-	5600 3300 5600 3500
-Wire Wire Line
 	4200 4900 4200 5300
 Wire Wire Line
@@
 	5100 5350 5100 5000
 Connection ~ 5100 5000
-Wire Wire Line
-	5500 5000 5600 5000
-Connection ~ 5600 5000
 Wire Wire Line
 	6000 5000 6100 5000
@@
 	7300 4800 7350 4800
 Connection ~ 6500 6100
-Wire Wire Line
-	5600 3800 5600 5000
 Wire Wire Line
 	6700 4700 6700 4800
@@
 	5100 5000 5200 5000
 Wire Wire Line
-	5600 5000 5700 5000
-Wire Wire Line
 	6100 5000 6200 5000
 Wire Wire Line
@@
 	1    0    0    -1
 $EndComp
-Connection ~ 5600 3300
 $Comp
 L Connector:TestPoint TP4
@@
 Connection ~ 9450 1450
 Connection ~ 9950 1450
+$Comp
+L Device:Jumper_NC_Small JP3
+U 1 1 5CBCB580
+P 5600 4000
+F 0 "JP3" H 5600 4212 50  0000 C CNN
+F 1 "VCA_IN" H 5600 4121 50  0000 C CNN
+F 2 "Connector_PinHeader_2.54mm:PinHeader_1x02_P2.54mm_Vertical" H 5600 4000 50  0001 C CNN
+F 3 "~" H 5600 4000 50  0001 C CNN
+	1    5600 4000
+	0    1    1    0
+$EndComp
+Connection ~ 5600 3300
+Wire Wire Line
+	5600 3300 5600 3450
+Wire Wire Line
+	5500 5000 5600 5000
+Wire Wire Line
+	5600 3750 5600 3900
+Wire Wire Line
+	5600 4100 5600 5000
+Connection ~ 5600 5000
+Wire Wire Line
+	5600 5000 5700 5000
 $EndSCHEMATC

Commit message: Just notes in some schematics
Other:
- note added: "NOTE: When building, consider this:\nC8 is 1nF in my prototype, and I \ncouldn’t see C11 at all. \nExperiment and listen."
Changed lines of the file:
@@
 Wire Wire Line
 	5600 5000 5700 5000
+Text Notes 6750 4150 0    50   ~ 0
+NOTE: When building, consider this:\nC8 is 1nF in my prototype, and I \ncouldn’t see C11 at all. \nExperiment and listen.
 $EndSCHEMATC
