File: pro3320/kicad_files/pro3320.sch (KiCad schematic (older format))
At the start: 86 parts, among them J1 RES_CV_IN, J2 AUDIO_IN, J3 FREQ_CV_IN, J4 EUROPOWER, J5 OUT_MAIN, J6 OUT_C, J7 OUT_B, J8 OUT_A, SW1 LP_HP_2, SW2 LP_HP_1, SW3 LP_HP_3, SW4 LP_HP_4, U1 TL074, U2 AS3320, U3 TL074

Commit message: pro3320: Start working on PCB
Parts:
- removed J1: RES_CV_IN, symbol pro3320-rescue:Audio-Jack-2
- removed J2: AUDIO_IN, symbol pro3320-rescue:Audio-Jack-2
- removed J3: FREQ_CV_IN, symbol pro3320-rescue:Audio-Jack-2
- removed J5: OUT_MAIN, symbol pro3320-rescue:Audio-Jack-2
- removed J6: OUT_C, symbol pro3320-rescue:Audio-Jack-2
- removed J7: OUT_B, symbol pro3320-rescue:Audio-Jack-2
- removed J8: OUT_A, symbol pro3320-rescue:Audio-Jack-2
- removed SW1: LP_HP_2, symbol pro3320-rescue:SW_3PDT
- removed SW3: LP_HP_3, symbol pro3320-rescue:SW_3PDT
- removed SW4: LP_HP_4, symbol pro3320-rescue:SW_3PDT
- added J1: RES_CV_IN, kicadlib:PJ301BM, symbol hakane:AudioJack_Mono_Switch
- added J2: AUDIO_IN, kicadlib:PJ301BM, symbol hakane:AudioJack_Mono_Switch
- added J3: FREQ_CV_IN, kicadlib:PJ301BM, symbol hakane:AudioJack_Mono_Switch
- added J5: OUT_MAIN, kicadlib:PJ301BM, symbol hakane:AudioJack_Mono_Switch
- added J6: OUT_3, kicadlib:PJ301BM, symbol hakane:AudioJack_Mono_Switch
- added J7: OUT_2, kicadlib:PJ301BM, symbol hakane:AudioJack_Mono_Switch
- added J8: OUT_1, kicadlib:PJ301BM, symbol hakane:AudioJack_Mono_Switch
- added R48: 68k, Resistor_THT:R_Axial_DIN0207_L6.3mm_D2.5mm_P7.62mm_Horizontal, symbol Device:R
- added SW1: LP_HP_CAP_2, kicadlib:DPDT_AS_SPDT_PUSH_SW, symbol Switch:SW_SPDT
- added SW3: LP_HP_2, kicadlib:DPDT_PUSH_SW, symbol pro3320-rescue:SW_DPDT_x2
- added SW4: LP_HP_CAP_3, kicadlib:DPDT_AS_SPDT_PUSH_SW, symbol Switch:SW_SPDT
- added SW5: LP_HP_3, kicadlib:DPDT_PUSH_SW, symbol pro3320-rescue:SW_DPDT_x2
- added SW6: LP_HP_CAP_4, kicadlib:DPDT_AS_SPDT_PUSH_SW, symbol Switch:SW_SPDT
- added SW7: LP_HP_4, kicadlib:DPDT_PUSH_SW, symbol pro3320-rescue:SW_DPDT_x2
- added TP1: OUT_STAGE_1, TestPoint:TestPoint_THTPad_3.0x3.0mm_Drill1.5mm, symbol Connector:TestPoint
- added TP2: OUT_STAGE_2, TestPoint:TestPoint_THTPad_3.0x3.0mm_Drill1.5mm, symbol Connector:TestPoint
- added TP3: OUT_STAGE_4, TestPoint:TestPoint_THTPad_3.0x3.0mm_Drill1.5mm, symbol Connector:TestPoint
- added TP4: OUT_STAGE_3, TestPoint:TestPoint_THTPad_3.0x3.0mm_Drill1.5mm, symbol Connector:TestPoint
- C1: value CP -> 2.2uF; footprint (none) -> Capacitor_THT:CP_Radial_D5.0mm_P2.00mm
- C10, C11, C6, C7, C8, C9: footprint (none) -> Capacitor_THT:C_Rect_L7.2mm_W3.5mm_P5.00mm_FKS2_FKP2_MKS2_MKP2
- C12, C13, C2, C3: footprint (none) -> Capacitor_THT:C_Rect_L7.0mm_W3.5mm_P5.00mm
- C14, C15, C16, C17, C4, C5: footprint (none) -> Capacitor_THT:CP_Radial_D5.0mm_P2.00mm
- D1, D2: footprint Diodes_THT:D_DO-41_SOD81_Horizontal_RM10 -> Diode_THT:D_DO-41_SOD81_P7.62mm_Horizontal
- J4: footprint (none) -> Connector_PinHeader_2.54mm:PinHeader_2x05_P2.54mm_Vertical
- R1, R10, R11, R12, R13, R14, R15, R16, R17, R18, R19, R2, R20, R21, R22, R23, R24, R25, R26, R27, R28, R29, R3, R30, R31, R32, R33, R34, R35, R36, R37, R38, R39, R4, R40, R41, R42, R43, R44, R45, R46, R47, R5, R6, R7, R8, R9: footprint (none) -> Resistor_THT:R_Axial_DIN0207_L6.3mm_D2.5mm_P7.62mm_Horizontal
- RV1, RV2, RV4, RV5: footprint (none) -> Potentiometer_THT:Potentiometer_Alps_RK09K_Single_Vertical
- RV3: value POT -> 100k; footprint (none) -> Potentiometer_THT:Potentiometer_Alps_RK09K_Single_Vertical
- SW2: footprint (none) -> kicadlib:DPDT_PUSH_SW
- U1, U3: footprint (none) -> Package_DIP:DIP-14_W7.62mm
- U2: footprint (none) -> Package_DIP:DIP-18_W7.62mm
Connections:
- wire segments 271 -> 307
- no-connect marks 7 -> 15
Other:
- note added: "NOTE: The 68k between pos input and\nGND is from ProOne – what does it do?\n"
- note added: "OR IS IT 10V p-p????\n-- Testable on PCB, breadboard not needed."
- note added: "TEST AT LEAST ONE HP/LP SWITCH? \nAND ONE SEPARATE OUTPUT?\n-- Or, assume it will be OK. If not, \njust don't mount the switches/outs."
- note added: "TEST RANGE OF FREQ CV POT\nTEST RANGE OF RES CV POT\n-- Testable on PCB, no need for breadboard.\n"
- note added: "TEST THESE OUTS\nTestable on PCB. First, don't connect at all, start with normal out."
- note added: "TEST THIS, REALLY UNSURE. ALL THREE COMPONENTS.\nTestable on PCB, breadboard not needed."
- note removed: "NOTE: ProOne has 68k between \npos input and GND – why?\n"
- note removed: "OR IS IT 10V p-p????\n"
- note removed: "TEST AT LEAST ONE HP/LP SWITCH? \nAND ONE SEPARATE OUTPUT?"
- note removed: "TEST RANGE OF FREQ CV POT\nTEST RANGE OF RES CV POT\n"
- note removed: "TEST THESE OUTS"
- note removed: "TEST THIS, REALLY UNSURE. ALL THREE COMPONENTS."

Commit message: pro3320: Abandon panel PCB
I tried having a PCB parallell to the panel, but it gets too
wide for my taste (and/or requires too much time and brain
activity in the PCB layout tool).

Will slim it down, having the PCB hanging on the pots, and
mounting the jacks on panel, the switches as well, having
to solder a LOT of cables. It will be hell, but I don't see
another way (except having two PCBs, layered, but that's too
much for me now).
Parts:
- C12, C13, C2, C3: value 300p -> 150p
- J1: value RES_CV_IN -> RES_CV
- J2: value AUDIO_IN -> IN
- J3: value FREQ_CV_IN -> FREQ_CV
- J5: value OUT_MAIN -> OUT
Other:
- note added: "NOTE: The 68k between pos input and\nGND is from ProOne – what does it do?\nAnd should the other outs have one as well?"
- note added: "NOTE: Using 150pF for filter capacitors, like ProOne.\nApparently, this raises the base frequency one octave."
- note removed: "NOTE: The 68k between pos input and\nGND is from ProOne – what does it do?\n"
Changed lines of the file:
@@
 P 4650 2600
 F 0 "C3" H 4675 2700 50  0000 L CNN
-F 1 "300p" H 4675 2500 50  0000 L CNN
+F 1 "150p" H 4675 2500 50  0000 L CNN
 F 2 "Capacitor_THT:C_Rect_L7.0mm_W3.5mm_P5.00mm" H 4688 2450 50  0001 C CNN
 F 3 "" H 4650 2600 50  0001 C CNN
@@
 P 4550 3450
 F 0 "C2" H 4575 3550 50  0000 L CNN
-F 1 "300p" V 4600 3200 50  0000 L CNN
+F 1 "150p" V 4600 3200 50  0000 L CNN
 F 2 "Capacitor_THT:C_Rect_L7.0mm_W3.5mm_P5.00mm" H 4588 3300 50  0001 C CNN
 F 3 "" H 4550 3450 50  0001 C CNN
@@
 P 6700 3650
 F 0 "C12" H 6725 3750 50  0000 L CNN
-F 1 "300p" V 6750 3400 50  0000 L CNN
+F 1 "150p" V 6750 3400 50  0000 L CNN
 F 2 "Capacitor_THT:C_Rect_L7.0mm_W3.5mm_P5.00mm" H 6738 3500 50  0001 C CNN
 F 3 "" H 6700 3650 50  0001 C CNN
@@
 P 6700 4650
 F 0 "C13" H 6725 4750 50  0000 L CNN
-F 1 "300p" H 6725 4550 50  0000 L CNN
+F 1 "150p" H 6725 4550 50  0000 L CNN
 F 2 "Capacitor_THT:C_Rect_L7.0mm_W3.5mm_P5.00mm" H 6738 4500 50  0001 C CNN
 F 3 "" H 6700 4650 50  0001 C CNN
@@
 $EndComp
 Text Notes 9500 350  0    60   ~ 0
-NOTE: The 68k between pos input and\nGND is from ProOne – what does it do?\n
+NOTE: The 68k between pos input and\nGND is from ProOne – what does it do?\nAnd should the other outs have one as well?
 $Comp
 L pro3320-rescue:R R27
@@
 P 750 1250
 F 0 "J1" H 754 1592 50  0000 C CNN
-F 1 "RES_CV_IN" H 754 1501 50  0000 C CNN
+F 1 "RES_CV" H 754 1501 50  0000 C CNN
 F 2 "kicadlib:PJ301BM" H 750 1250 50  0001 C CNN
 F 3 "~" H 750 1250 50  0001 C CNN
@@
 P 750 2000
 F 0 "J2" H 754 2342 50  0000 C CNN
-F 1 "AUDIO_IN" H 754 2251 50  0000 C CNN
+F 1 "IN" H 754 2251 50  0000 C CNN
 F 2 "kicadlib:PJ301BM" H 750 2000 50  0001 C CNN
 F 3 "~" H 750 2000 50  0001 C CNN
@@
 P 750 5950
 F 0 "J3" H 754 6292 50  0000 C CNN
-F 1 "FREQ_CV_IN" H 754 6201 50  0000 C CNN
+F 1 "FREQ_CV" H 754 6201 50  0000 C CNN
 F 2 "kicadlib:PJ301BM" H 750 5950 50  0001 C CNN
 F 3 "~" H 750 5950 50  0001 C CNN
@@
 P 10900 1100
 F 0 "J5" H 10900 1350 50  0000 R CNN
-F 1 "OUT_MAIN" H 11000 900 50  0000 R CNN
+F 1 "OUT" H 11000 900 50  0000 R CNN
 F 2 "kicadlib:PJ301BM" H 10900 1100 50  0001 C CNN
 F 3 "~" H 10900 1100 50  0001 C CNN
@@
 U 1 1 5CE1A2F8
 P 9150 1200
-F 0 "R48" H 9000 1150 50  0000 L CNN
+F 0 "R48" V 9050 1100 50  0000 L CNN
 F 1 "68k" V 9150 1150 50  0000 L CNN
 F 2 "Resistor_THT:R_Axial_DIN0207_L6.3mm_D2.5mm_P7.62mm_Horizontal" V 9080 1200 50  0001 C CNN
@@
 Wire Wire Line
 	3650 6300 8700 6300
+Text Notes 1950 7550 0    50   ~ 0
+NOTE: Using 150pF for filter capacitors, like ProOne.\nApparently, this raises the base frequency one octave.
 $EndSCHEMATC

Commit message: pro3320: First messy PCB attempt
Parts:
- removed C10: 100nF, Capacitor_THT:C_Rect_L7.2mm_W3.5mm_P5.00mm_FKS2_FKP2_MKS2_MKP2, symbol pro3320-rescue:C
- removed C15, C16, C17: 2.2uF, Capacitor_THT:CP_Radial_D5.0mm_P2.00mm, symbol pro3320-rescue:CP
- removed J7: OUT_2, kicadlib:PJ301BM, symbol hakane:AudioJack_Mono_Switch
- removed J8: OUT_1, kicadlib:PJ301BM, symbol hakane:AudioJack_Mono_Switch
- removed R35: 100k, Resistor_THT:R_Axial_DIN0207_L6.3mm_D2.5mm_P7.62mm_Horizontal, symbol pro3320-rescue:R
- removed R37, R38, R39: 240k, Resistor_THT:R_Axial_DIN0207_L6.3mm_D2.5mm_P7.62mm_Horizontal, symbol pro3320-rescue:R
- removed R41, R42, R43, R45, R46, R47: 2.2k, Resistor_THT:R_Axial_DIN0207_L6.3mm_D2.5mm_P7.62mm_Horizontal, symbol pro3320-rescue:R
- removed SW1: LP_HP_CAP_2, kicadlib:DPDT_AS_SPDT_PUSH_SW, symbol Switch:SW_SPDT
- removed SW3: LP_HP_2, kicadlib:DPDT_PUSH_SW, symbol pro3320-rescue:SW_DPDT_x2
- removed SW4: LP_HP_CAP_3, kicadlib:DPDT_AS_SPDT_PUSH_SW, symbol Switch:SW_SPDT
- removed SW5: LP_HP_3, kicadlib:DPDT_PUSH_SW, symbol pro3320-rescue:SW_DPDT_x2
- removed SW6: LP_HP_CAP_4, kicadlib:DPDT_AS_SPDT_PUSH_SW, symbol Switch:SW_SPDT
- removed SW7: LP_HP_4, kicadlib:DPDT_PUSH_SW, symbol pro3320-rescue:SW_DPDT_x2
- removed U3: TL074, Package_DIP:DIP-14_W7.62mm, symbol pro3320-rescue:TL074
- added C10: 2.2uF, Capacitor_THT:CP_Radial_D5.0mm_P2.00mm, symbol pro3320-rescue:CP
- added C15: 100nF, Capacitor_THT:C_Rect_L7.2mm_W3.5mm_P5.00mm_FKS2_FKP2_MKS2_MKP2, symbol pro3320-rescue:C
- added JP1: OPT_OUT2, Connector_PinHeader_2.54mm:PinHeader_1x02_P2.54mm_Vertical, symbol Device:Jumper
- added SW1: LPHP2, Connector_PinHeader_2.54mm:PinHeader_1x09_P2.54mm_Vertical, symbol hakane:SW_3PDT
- added SW3: LPHP3, Connector_PinHeader_2.54mm:PinHeader_1x09_P2.54mm_Vertical, symbol hakane:SW_3PDT
- added SW4: LPHP4, Connector_PinHeader_2.54mm:PinHeader_1x09_P2.54mm_Vertical, symbol hakane:SW_3PDT
- added U3: TL072, Package_DIP:DIP-8_W7.62mm, symbol Amplifier_Operational:TL072
- J1, J2, J3, J5: footprint kicadlib:PJ301BM -> Connector_PinHeader_2.54mm:PinHeader_1x03_P2.54mm_Vertical
- J6: value OUT_3 -> OUT2; footprint kicadlib:PJ301BM -> Connector_PinHeader_2.54mm:PinHeader_1x03_P2.54mm_Vertical
- R34: value 100k -> 240k
- RV1, RV2, RV3, RV4, RV5: footprint Potentiometer_THT:Potentiometer_Alps_RK09K_Single_Vertical -> Potentiometer_THT:Potentiometer_Alps_RK097_Single_Horizontal
- SW2: value LP_HP_1 -> LPHP1; footprint kicadlib:DPDT_PUSH_SW -> Connector_PinHeader_2.54mm:PinHeader_1x06_P2.54mm_Vertical
- TP1, TP2: footprint TestPoint:TestPoint_THTPad_3.0x3.0mm_Drill1.5mm -> TestPoint:TestPoint_THTPad_2.0x2.0mm_Drill1.0mm
- TP3: renamed from TP4; footprint TestPoint:TestPoint_THTPad_3.0x3.0mm_Drill1.5mm -> TestPoint:TestPoint_THTPad_2.0x2.0mm_Drill1.0mm
- TP4: renamed from TP3; footprint TestPoint:TestPoint_THTPad_3.0x3.0mm_Drill1.5mm -> TestPoint:TestPoint_THTPad_2.0x2.0mm_Drill1.0mm
Connections:
- wire segments 307 -> 273
- no-connect marks 15 -> 12
Other:
- note added: "Optional untested extra output, not in the PCB. \nPut it in because a TL072 takes no more room than \na TL071, so if one wants it, it’s there (for anything)."
- note removed: "It would be really nice to have insert jacks between \nstages. Although I think there is a slight risk that the \ninputs may disturb (destroy?) the IC, and also – it is \ndesigned to work like a chain... \nOn the other hand, it would be interesting to know \nwhat that would sound like. :-)"
- note removed: "TEST THESE OUTS\nTestable on PCB. First, don't connect at all, start with normal out."
- moved on the sheet: C4, C5, C6, C7, C8, C9, D1, D2, J4, TP1, TP2, TP3

Commit message: pro3320: Finish PCB routing
It's not pretty, but will hopefully work.
There is something missing in my layout knowledge,I believe;
it feels like a better layout would make routing easier.
Whatevs.
Parts:
- J1, J2, J3, J5, J6: footprint Connector_PinHeader_2.54mm:PinHeader_1x03_P2.54mm_Vertical -> Connector_PinHeader_2.54mm:PinHeader_1x02_P2.54mm_Vertical; symbol hakane:AudioJack_Mono_Switch -> hakane:AudioJack_Mono_No_Switch
Connections:
- no-connect marks 12 -> 7
Changed lines of the file:
@@
 Wire Wire Line
 	950  1250 1450 1250
-NoConn ~ 950  1350
-$Comp
-L hakane:AudioJack_Mono_Switch J1
+$Comp
+L hakane:AudioJack_Mono_No_Switch J1
 U 1 1 5CC04472
 P 750 1250
 F 0 "J1" H 754 1592 50  0000 C CNN
 F 1 "RES_CV" H 754 1501 50  0000 C CNN
-F 2 "Connector_PinHeader_2.54mm:PinHeader_1x03_P2.54mm_Vertical" H 750 1250 50  0001 C CNN
+F 2 "Connector_PinHeader_2.54mm:PinHeader_1x02_P2.54mm_Vertical" H 750 1250 50  0001 C CNN
 F 3 "~" H 750 1250 50  0001 C CNN
 	1    750  1250
@@
 $EndComp
 $Comp
-L hakane:AudioJack_Mono_Switch J2
+L hakane:AudioJack_Mono_No_Switch J2
 U 1 1 5CC04EC0
 P 750 2000
 F 0 "J2" H 754 2342 50  0000 C CNN
 F 1 "IN" H 754 2251 50  0000 C CNN
-F 2 "Connector_PinHeader_2.54mm:PinHeader_1x03_P2.54mm_Vertical" H 750 2000 50  0001 C CNN
+F 2 "Connector_PinHeader_2.54mm:PinHeader_1x02_P2.54mm_Vertical" H 750 2000 50  0001 C CNN
 F 3 "~" H 750 2000 50  0001 C CNN
 	1    750  2000
@@
 Wire Wire Line
 	950  2000 1050 2000
-NoConn ~ 950  2100
 $Comp
 L pro3320-rescue:GND #PWR041
@@
 	1000 950  1000 1150
 $Comp
-L hakane:AudioJack_Mono_Switch J3
+L hakane:AudioJack_Mono_No_Switch J3
 U 1 1 5CC594FC
 P 750 5950
 F 0 "J3" H 754 6292 50  0000 C CNN
 F 1 "FREQ_CV" H 754 6201 50  0000 C CNN
-F 2 "Connector_PinHeader_2.54mm:PinHeader_1x03_P2.54mm_Vertical" H 750 5950 50  0001 C CNN
+F 2 "Connector_PinHeader_2.54mm:PinHeader_1x02_P2.54mm_Vertical" H 750 5950 50  0001 C CNN
 F 3 "~" H 750 5950 50  0001 C CNN
 	1    750  5950
@@
 Wire Wire Line
 	950  5950 1300 5950
-NoConn ~ 950  6050
-$Comp
-L hakane:AudioJack_Mono_Switch J5
+$Comp
+L hakane:AudioJack_Mono_No_Switch J5
 U 1 1 5CDD4C87
 P 10900 1100
 F 0 "J5" H 10900 1350 50  0000 R CNN
 F 1 "OUT" H 11000 900 50  0000 R CNN
-F 2 "Connector_PinHeader_2.54mm:PinHeader_1x03_P2.54mm_Vertical" H 10900 1100 50  0001 C CNN
+F 2 "Connector_PinHeader_2.54mm:PinHeader_1x02_P2.54mm_Vertical" H 10900 1100 50  0001 C CNN
 F 3 "~" H 10900 1100 50  0001 C CNN
 	1    10900 1100
 	-1   0    0    -1
 $EndComp
-NoConn ~ 10700 1200
 Wire Wire Line
 	10700 1000 10650 1000
@@
 Optional untested extra output, not in the PCB. \nPut it in because a TL072 takes no more room than \na TL071, so if one wants it, it’s there (for anything).
 $Comp
-L hakane:AudioJack_Mono_Switch J6
+L hakane:AudioJack_Mono_No_Switch J6
 U 1 1 5CD970CB
 P 10900 4950
 F 0 "J6" H 10900 5200 50  0000 R CNN
 F 1 "OUT2" H 11000 4750 50  0000 R CNN
-F 2 "Connector_PinHeader_2.54mm:PinHeader_1x03_P2.54mm_Vertical" H 10900 4950 50  0001 C CNN
+F 2 "Connector_PinHeader_2.54mm:PinHeader_1x02_P2.54mm_Vertical" H 10900 4950 50  0001 C CNN
 F 3 "~" H 10900 4950 50  0001 C CNN
 	1    10900 4950
@@
 Wire Wire Line
 	10650 4850 10700 4850
-NoConn ~ 10700 5050
 $Comp
 L Amplifier_Operational:TL072 U3

Commit message: pro3320: Add logo to PCB
Also, polishing the PCB and schematic a wee bit.
Faced with the choice, what would you say?
Parts:
- TP1: value OUT_STAGE_1 -> OP1
- TP2: value OUT_STAGE_2 -> OP2
- TP3: value OUT_STAGE_3 -> OP3
- TP4: value OUT_STAGE_4 -> OP4
Other:
- note added: "A"
- note added: "A VCF built on the CEM3320,based on its data sheet reference \nimplementations, and a bit of inspiration from the ProOne.\n\nRev. A in a severe prototype state."
- note added: "April 16, 2019"
- note added: "pro3320 vcf\n"
Changed lines of the file:
@@
 P 9500 6050
 F 0 "TP1" H 9558 6170 50  0000 L CNN
-F 1 "OUT_STAGE_1" H 9558 6079 50  0000 L CNN
+F 1 "OP1" H 9558 6079 50  0000 L CNN
 F 2 "TestPoint:TestPoint_THTPad_2.0x2.0mm_Drill1.0mm" H 9700 6050 50  0001 C CNN
 F 3 "~" H 9700 6050 50  0001 C CNN
@@
 P 8100 6050
 F 0 "TP2" H 8158 6170 50  0000 L CNN
-F 1 "OUT_STAGE_2" H 8158 6079 50  0000 L CNN
+F 1 "OP2" H 8158 6079 50  0000 L CNN
 F 2 "TestPoint:TestPoint_THTPad_2.0x2.0mm_Drill1.0mm" H 8300 6050 50  0001 C CNN
 F 3 "~" H 8300 6050 50  0001 C CNN
@@
 P 8600 3900
 F 0 "TP3" H 8658 4020 50  0000 L CNN
-F 1 "OUT_STAGE_3" H 8658 3929 50  0000 L CNN
+F 1 "OP3" H 8658 3929 50  0000 L CNN
 F 2 "TestPoint:TestPoint_THTPad_2.0x2.0mm_Drill1.0mm" H 8800 3900 50  0001 C CNN
 F 3 "~" H 8800 3900 50  0001 C CNN
@@
 P 8150 1350
 F 0 "TP4" H 8350 1500 50  0000 R CNN
-F 1 "OUT_STAGE_4" H 8700 1400 50  0000 R CNN
+F 1 "OP4" H 8700 1400 50  0000 R CNN
 F 2 "TestPoint:TestPoint_THTPad_2.0x2.0mm_Drill1.0mm" H 8350 1350 50  0001 C CNN
 F 3 "~" H 8350 1350 50  0001 C CNN
@@
 Wire Wire Line
 	6250 6800 5950 6800
+Wire Notes Line
+	8800 5700 11150 5700
+Wire Notes Line
+	11150 5700 11150 4200
+Wire Notes Line
+	11150 4200 8800 4200
+Wire Notes Line
+	8800 4200 8800 5700
+Text Notes 8050 7000 0    50   ~ 0
+A VCF built on the CEM3320,based on its data sheet reference \nimplementations, and a bit of inspiration from the ProOne.\n\nRev. A in a severe prototype state.
+Text Notes 7500 7500 0    50   ~ 0
+pro3320 vcf\n
+Text Notes 10650 7650 0    50   ~ 0
+A
+Text Notes 8150 7650 0    50   ~ 0
+April 16, 2019
 $EndSCHEMATC

Commit message: pro3320: Fix wrong direction of pots
Changed lines of the file:
@@
 F 3 "" H 1450 1450 50  0001 C CNN
 	1    1450 1450
-	1    0    0    -1
+	1    0    0    1
 $EndComp
 Text Notes 550  4750 0    60   ~ 0
@@
 F 3 "" H 1300 5550 50  0001 C CNN
 	1    1300 5550
-	1    0    0    -1
+	1    0    0    1
 $EndComp
 $Comp
@@
 F 3 "" H 1300 6150 50  0001 C CNN
 	1    1300 6150
-	1    0    0    -1
+	1    0    0    1
 $EndComp
 $Comp
@@
 F 3 "" H 1450 2200 50  0001 C CNN
 	1    1450 2200
-	1    0    0    -1
+	1    0    0    1
 $EndComp
 $Comp
@@
 F 3 "" H 2150 900 50  0001 C CNN
 	1    2150 900
-	1    0    0    -1
-$EndComp
-$Comp
+	1    0    0    1
+$EndComp
+$Comp

Commit message: Just notes in some schematics
Other:
- note added: "Normal level in should \nbe about 10V p-p, but \nadding a bit more gain \nto the amp, so that weak\nsignals can have a go \n(and to see whether \nthat kind of distortion \nagrees with the VCF)."
- note removed: "Normal level in should \nbe about +/-10V, but \nadding a bit more gain \nto the amp, so that weak\nsignals can have a go \n(and to see whether \nthat kind of distortion \nagrees with the VCF)."
- note removed: "OR IS IT 10V p-p????\n-- Testable on PCB, breadboard not needed."
Changed lines of the file:
@@
 $EndComp
 Text Notes 550  3350 0    60   ~ 0
-Normal level in should \nbe about +/-10V, but \nadding a bit more gain \nto the amp, so that weak\nsignals can have a go \n(and to see whether \nthat kind of distortion \nagrees with the VCF).
+Normal level in should \nbe about 10V p-p, but \nadding a bit more gain \nto the amp, so that weak\nsignals can have a go \n(and to see whether \nthat kind of distortion \nagrees with the VCF).
 $Comp
 L pro3320-rescue:R R9
@@
 	1    0    0    -1
 $EndComp
-Text Notes 350  3350 1    60   ~ 0
-OR IS IT 10V p-p????\n-- Testable on PCB, breadboard not needed.
 Wire Wire Line
 	4700 2850 4650 2850

Commit message: pro3320: Update docs and some component values
Parts:
- R15, R25, R30: value 220k -> 200k
Changed lines of the file:
@@
 P 3450 4400
 F 0 "R15" V 3530 4400 50  0000 C CNN
-F 1 "220k" V 3450 4400 50  0000 C CNN
+F 1 "200k" V 3450 4400 50  0000 C CNN
 F 2 "Resistor_THT:R_Axial_DIN0207_L6.3mm_D2.5mm_P7.62mm_Horizontal" V 3380 4400 50  0001 C CNN
 F 3 "" H 3450 4400 50  0001 C CNN
@@
 P 6350 5750
 F 0 "R25" V 6430 5750 50  0000 C CNN
-F 1 "220k" V 6350 5750 50  0000 C CNN
+F 1 "200k" V 6350 5750 50  0000 C CNN
 F 2 "Resistor_THT:R_Axial_DIN0207_L6.3mm_D2.5mm_P7.62mm_Horizontal" V 6280 5750 50  0001 C CNN
 F 3 "" H 6350 5750 50  0001 C CNN
@@
 P 7350 2500
 F 0 "R30" V 7430 2500 50  0000 C CNN
-F 1 "220k" V 7350 2500 50  0000 C CNN
+F 1 "200k" V 7350 2500 50  0000 C CNN
 F 2 "Resistor_THT:R_Axial_DIN0207_L6.3mm_D2.5mm_P7.62mm_Horizontal" V 7280 2500 50  0001 C CNN
 F 3 "" H 7350 2500 50  0001 C CNN
