File: minidrum-77/kicad_files/minidrum-77.sch (KiCad schematic (older format))
At the start: 19 parts, among them J1 AudioJack2_Ground, J2 AudioJack2_Ground

Commit message: Add coil jumper on DR-77/78
Parts:
- added JP1: ALT_COIL, symbol Jumper:Jumper_3_Bridged12
- D1: footprint (none) -> Diode_THT:D_DO-35_SOD27_P7.62mm_Horizontal
Connections:
- wire segments 57 -> 58
- no-connect marks 0 -> 1
Other:
- note added: "A"
- note added: "DR-77/78"
- note added: "DR-77/78\nClave/Rimshot/BD/etc. sounds from TR-77 and CR-78"
- note added: "For C1 on the TR-77 sounds: instead of a jumper,\ntry 27nF as on the CR-78 – is there a difference?"
- note added: "JP1 can be used to connect a\ndifferent coil, e.g. via external jack."
- note added: "January 26, 2019"
- note removed: "For C1 on the TR-77 sounds — instead of a jumper,\nconsider using 27nF as on the CR-77"

Commit message: Add coil footprint, update DR-77/78
Parts:
- J1, J2: footprint (none) -> MusicThingModular:NV-PJ3410_SOCKET_MONO
- JP1: footprint (none) -> Connector_PinHeader_2.54mm:PinHeader_1x03_P2.54mm_Vertical
- L1: footprint (none) -> kicadlib:CoilC-1X
- R1, R2, R3, R4, R5: footprint (none) -> MusicThingModular:10MM_RESISTOR
Other:
- note added: "CR-78 Claves\n—————————\nC1: 27nF\nR1: 270k\nC2: NC\nD1: (see note)\nR2: 2.2M\nR3: 47k\nR4: NC\nC3: 4.7 nF\nC4: 2.2 nF\nC5: 4.7 nF\nC6: NC\nL1: 700 mH\nC7: 250 pF\nC8: 5.6 nF\nC9: 1 nF\nR5: NC\nC10: NC\n"
- note added: "CR-78 Rim Shot\n—————————\nC1: 27nF\nR1: 270k\nC2: NC\nD1: (see note)\nR2: NC\nR3: 47k\nR4: 47k\nC3: NC\nC4: NC\nC5: 1.5 nF\nC6: 15 nF\nL1: 700 mH\nC7: 470 pF\nC8: NC\nC9: NC\nR5: 0 (jumper)\nC10: NC"
- note added: "Inductors at Mouser: \nC-1X 15H (Triad Magnetics)\nC-85X 1.5H (Triad Magnetics)"
- note added: "NOTE: For C1 on the TR-77 sounds: instead of a jumper,\ntry 27nF as on the CR-78 – is there a difference?"
- note added: "NOTE: The coil values for the listed CR-78 voices are guessed:\nhttp://electro-music.com/forum/post-420004.html#420004"
- note added: "NOTE: The diode is most likely not that important.\nI think I’ll go for a BAT-42, since it has low voltage\ndrop; I’m sure a standard 1N4148 will do as well.\nIf you want the original, check the original schematics. :-)"
- note added: "TR-77 Bass Drum\n—————————\nC1: 0 (jumper)\nR1: NC\nC2: 4.7 nF\nD1: (see note)\nR2: 4.7M\nR3: 33k\nR4: NC\nC3: 56 nF\nC4: 33 nF\nC5: 220 nF\nC6: 1 nF\nL1: 16 H (!)\nC7: 33 nF\nC8: 100 nF\nC9: NC\nR5: 10 k\nC10: 220 nF"
- note added: "TR-77 Claves\n—————————\nC1: 0 (jumper)\nR1: NC\nC2: 4.7 nF\nD1: (see note)\nR2: 4.7M\nR3: 56k\nR4: NC\nC3: 4.7 nF\nC4: 1 nF\nC5: 4.7 nF\nC6: NC\nL1: 700 mH\nC7: 1.5 nF\nC8: 5.6 nF\nC9: 2.2 nF\nR5: NC\nC10: NC"
- note added: "TR-77 Rim Shot\n—————————\nC1: 0 (jumper)\nR1: NC\nC2: 4.7 nF\nD1: (see note)\nR2: 4.7M\nR3: 100k\nR4: 47k\nC3: NC\nC4: 0 (jumper)\nC5: 27 nF\nC6: NC\nL1: 700 mH\nC7: 1 nF\nC8: NC\nC9: NC\nR5: 0 (jumper)\nC10: NC\n"
- note removed: "CR-78 Claves\n—————————\nC1: 27nF\nR1: 270k\nC2: NC\nD1: ???????\nR2: 2.2M\nR3: 47k\nR4: NC\nC3: 4.7 nF\nC4: 2.2 nF\nC5: 4.7 nF\nC6: NC\nL1: ??? mH\nC7: 250 pF\nC8: 5.6 nF\nC9: 1 nF\nR5: NC\nC10: NC\n"
- note removed: "CR-78 Rim Shot\n—————————\nC1: 27nF\nR1: 270k\nC2: NC\nD1: ???????\nR2: NC\nR3: 47k\nR4: 47k\nC3: NC\nC4: NC\nC5: 1.5 nF\nC6: 15 nF\nL1: ??? mH\nC7: 470 pF\nC8: NC\nC9: NC\nR5: 0 (jumper)\nC10: NC"
- note removed: "For C1 on the TR-77 sounds: instead of a jumper,\ntry 27nF as on the CR-78 – is there a difference?"
- note removed: "TR-77 Bass Drum\n—————————\nC1: 0 (jumper)\nR1: NC\nC2: 4.7 nF\nD1: ???????\nR2: 4.7M\nR3: 33k\nR4: NC\nC3: 56 nF\nC4: 33 nF\nC5: 220 nF\nC6: 1 nF\nL1: 16 H (!)\nC7: 33 nF\nC8: 100 nF\nC9: NC\nR5: 10 k\nC10: 220 nF"
- note removed: "TR-77 Claves\n—————————\nC1: 0 (jumper)\nR1: NC\nC2: 4.7 nF\nD1: ???????\nR2: 4.7M\nR3: 56k\nR4: NC\nC3: 4.7 nF\nC4: 1 nF\nC5: 4.7 nF\nC6: NC\nL1: 700 mH\nC7: 1.5 nF\nC8: 5.6 nF\nC9: 2.2 nF\nR5: NC\nC10: NC"
- note removed: "TR-77 Rim Shot\n—————————\nC1: 0 (jumper)\nR1: NC\nC2: 4.7 nF\nD1: ???????\nR2: 4.7M\nR3: 100k\nR4: 47k\nC3: NC\nC4: 0 (jumper)\nC5: 27 nF\nC6: NC\nL1: 700 mH\nC7: 1 nF\nC8: NC\nC9: NC\nR5: 0 (jumper)\nC10: NC\n"
Changed lines of the file:
@@
 F 0 "J1" H 1718 2479 50  0000 R CNN
 F 1 "AudioJack2_Ground" H 1718 2570 50  0000 R CNN
-F 2 "" H 1950 2500 50  0001 C CNN
+F 2 "MusicThingModular:NV-PJ3410_SOCKET_MONO" H 1950 2500 50  0001 C CNN
 F 3 "~" H 1950 2500 50  0001 C CNN
 	1    1950 2500
@@
 F 0 "J2" H 9167 2479 50  0000 R CNN
 F 1 "AudioJack2_Ground" H 9167 2570 50  0000 R CNN
-F 2 "" H 9400 2500 50  0001 C CNN
+F 2 "MusicThingModular:NV-PJ3410_SOCKET_MONO" H 9400 2500 50  0001 C CNN
 F 3 "~" H 9400 2500 50  0001 C CNN
 	1    9400 2500
@@
 F 0 "R1" H 3120 2946 50  0000 L CNN
 F 1 "R" H 3120 2855 50  0000 L CNN
-F 2 "" V 2980 2900 50  0001 C CNN
+F 2 "MusicThingModular:10MM_RESISTOR" V 2980 2900 50  0001 C CNN
 F 3 "~" H 3050 2900 50  0001 C CNN
 	1    3050 2900
@@
 F 0 "R2" H 4220 2946 50  0000 L CNN
 F 1 "R" H 4220 2855 50  0000 L CNN
-F 2 "" V 4080 2900 50  0001 C CNN
+F 2 "MusicThingModular:10MM_RESISTOR" V 4080 2900 50  0001 C CNN
 F 3 "~" H 4150 2900 50  0001 C CNN
 	1    4150 2900
@@
 F 0 "R3" V 4293 2500 50  0000 C CNN
 F 1 "R" V 4384 2500 50  0000 C CNN
-F 2 "" V 4430 2500 50  0001 C CNN
+F 2 "MusicThingModular:10MM_RESISTOR" V 4430 2500 50  0001 C CNN
 F 3 "~" H 4500 2500 50  0001 C CNN
 	1    4500 2500
@@
 F 0 "R4" H 4920 2946 50  0000 L CNN
 F 1 "R" H 4920 2855 50  0000 L CNN
-F 2 "" V 4780 2900 50  0001 C CNN
+F 2 "MusicThingModular:10MM_RESISTOR" V 4780 2900 50  0001 C CNN
 F 3 "~" H 4850 2900 50  0001 C CNN
 	1    4850 2900
@@
 F 0 "L1" H 6803 2996 50  0000 L CNN
 F 1 "L" H 6803 2905 50  0000 L CNN
-F 2 "" H 6750 2950 50  0001 C CNN
+F 2 "kicadlib:CoilC-1X" H 6750 2950 50  0001 C CNN
 F 3 "~" H 6750 2950 50  0001 C CNN
 	1    6750 2950
@@
 F 0 "R5" V 8143 2500 50  0000 C CNN
 F 1 "R" V 8234 2500 50  0000 C CNN
-F 2 "" V 8280 2500 50  0001 C CNN
+F 2 "MusicThingModular:10MM_RESISTOR" V 8280 2500 50  0001 C CNN
 F 3 "~" H 8350 2500 50  0001 C CNN
 	1    8350 2500
@@
 Connection ~ 3050 2500
 Text Notes 2250 5750 0    59   ~ 0
-CR-78 Claves\n—————————\nC1: 27nF\nR1: 270k\nC2: NC\nD1: ???????\nR2: 2.2M\nR3: 47k\nR4: NC\nC3: 4.7 nF\nC4: 2.2 nF\nC5: 4.7 nF\nC6: NC\nL1: ??? mH\nC7: 250 pF\nC8: 5.6 nF\nC9: 1 nF\nR5: NC\nC10: NC\n
+CR-78 Claves\n—————————\nC1: 27nF\nR1: 270k\nC2: NC\nD1: (see note)\nR2: 2.2M\nR3: 47k\nR4: NC\nC3: 4.7 nF\nC4: 2.2 nF\nC5: 4.7 nF\nC6: NC\nL1: 700 mH\nC7: 250 pF\nC8: 5.6 nF\nC9: 1 nF\nR5: NC\nC10: NC\n
 Text Notes 3150 5750 0    59   ~ 0
-CR-78 Rim Shot\n—————————\nC1: 27nF\nR1: 270k\nC2: NC\nD1: ???????\nR2: NC\nR3: 47k\nR4: 47k\nC3: NC\nC4: NC\nC5: 1.5 nF\nC6: 15 nF\nL1: ??? mH\nC7: 470 pF\nC8: NC\nC9: NC\nR5: 0 (jumper)\nC10: NC
+CR-78 Rim Shot\n—————————\nC1: 27nF\nR1: 270k\nC2: NC\nD1: (see note)\nR2: NC\nR3: 47k\nR4: 47k\nC3: NC\nC4: NC\nC5: 1.5 nF\nC6: 15 nF\nL1: 700 mH\nC7: 470 pF\nC8: NC\nC9: NC\nR5: 0 (jumper)\nC10: NC
 Text Notes 4050 5750 0    59   ~ 0
-TR-77 Claves\n—————————\nC1: 0 (jumper)\nR1: NC\nC2: 4.7 nF\nD1: ???????\nR2: 4.7M\nR3: 56k\nR4: NC\nC3: 4.7 nF\nC4: 1 nF\nC5: 4.7 nF\nC6: NC\nL1: 700 mH\nC7: 1.5 nF\nC8: 5.6 nF\nC9: 2.2 nF\nR5: NC\nC10: NC
+TR-77 Claves\n—————————\nC1: 0 (jumper)\nR1: NC\nC2: 4.7 nF\nD1: (see note)\nR2: 4.7M\nR3: 56k\nR4: NC\nC3: 4.7 nF\nC4: 1 nF\nC5: 4.7 nF\nC6: NC\nL1: 700 mH\nC7: 1.5 nF\nC8: 5.6 nF\nC9: 2.2 nF\nR5: NC\nC10: NC
 Text Notes 4950 5750 0    59   ~ 0
-TR-77 Rim Shot\n—————————\nC1: 0 (jumper)\nR1: NC\nC2: 4.7 nF\nD1: ???????\nR2: 4.7M\nR3: 100k\nR4: 47k\nC3: NC\nC4: 0 (jumper)\nC5: 27 nF\nC6: NC\nL1: 700 mH\nC7: 1 nF\nC8: NC\nC9: NC\nR5: 0 (jumper)\nC10: NC\n
+TR-77 Rim Shot\n—————————\nC1: 0 (jumper)\nR1: NC\nC2: 4.7 nF\nD1: (see note)\nR2: 4.7M\nR3: 100k\nR4: 47k\nC3: NC\nC4: 0 (jumper)\nC5: 27 nF\nC6: NC\nL1: 700 mH\nC7: 1 nF\nC8: NC\nC9: NC\nR5: 0 (jumper)\nC10: NC\n
 Text Notes 5850 5750 0    59   ~ 0
-TR-77 Bass Drum\n—————————\nC1: 0 (jumper)\nR1: NC\nC2: 4.7 nF\nD1: ???????\nR2: 4.7M\nR3: 33k\nR4: NC\nC3: 56 nF\nC4: 33 nF\nC5: 220 nF\nC6: 1 nF\nL1: 16 H (!)\nC7: 33 nF\nC8: 100 nF\nC9: NC\nR5: 10 k\nC10: 220 nF
+TR-77 Bass Drum\n—————————\nC1: 0 (jumper)\nR1: NC\nC2: 4.7 nF\nD1: (see note)\nR2: 4.7M\nR3: 33k\nR4: NC\nC3: 56 nF\nC4: 33 nF\nC5: 220 nF\nC6: 1 nF\nL1: 16 H (!)\nC7: 33 nF\nC8: 100 nF\nC9: NC\nR5: 10 k\nC10: 220 nF
 Text Notes 4050 6100 0    59   ~ 0
-For C1 on the TR-77 sounds: instead of a jumper,\ntry 27nF as on the CR-78 – is there a difference?
+NOTE: For C1 on the TR-77 sounds: instead of a jumper,\ntry 27nF as on the CR-78 – is there a difference?
 Wire Wire Line
 	9100 2600 9100 3300
@@
 F 0 "JP1" H 7000 2862 50  0000 C CNN
 F 1 "ALT_COIL" H 7000 2953 50  0000 C CNN
-F 2 "" H 7000 2750 50  0001 C CNN
+F 2 "Connector_PinHeader_2.54mm:PinHeader_1x03_P2.54mm_Vertical" H 7000 2750 50  0001 C CNN
 F 3 "~" H 7000 2750 50  0001 C CNN
 	1    7000 2750
@@
 Text Notes 10650 7650 0    50   ~ 0
 A
+Text Notes 4050 6400 0    59   ~ 0
+NOTE: The coil values for the listed CR-78 voices are guessed:\nhttp://electro-music.com/forum/post-420004.html#420004
+Text Notes 4050 6900 0    59   ~ 0
+NOTE: The diode is most likely not that important.\nI think I’ll go for a BAT-42, since it has low voltage\ndrop; I’m sure a standard 1N4148 will do as well.\nIf you want the original, check the original schematics. :-)
+Text Notes 2250 6550 0    50   ~ 0
+Inductors at Mouser: \nC-1X    15H (Triad Magnetics)\nC-85X  1.5H (Triad Magnetics)
 $EndSCHEMATC

Commit message: First revision of DR-77/78 PCB
Parts:
- removed J1, J2: AudioJack2_Ground, MusicThingModular:NV-PJ3410_SOCKET_MONO, symbol Connector:AudioJack2_Ground
- added J1: TRIG_IN, kicadlib:PJ301BM, symbol hakane:AudioJack_Mono_Switch
- added J2: AUDIO_OUT, kicadlib:PJ301BM, symbol hakane:AudioJack_Mono_Switch
- R1, R2, R3, R4, R5: footprint MusicThingModular:10MM_RESISTOR -> Resistor_THT:R_Axial_DIN0207_L6.3mm_D2.5mm_P10.16mm_Horizontal
Connections:
- no-connect marks 1 -> 3
Changed lines of the file:
@@
 $EndDescr
-$Comp
-L Connector:AudioJack2_Ground J1
-U 1 1 5BCF78C7
-P 1950 2500
-F 0 "J1" H 1718 2479 50  0000 R CNN
-F 1 "AudioJack2_Ground" H 1718 2570 50  0000 R CNN
-F 2 "MusicThingModular:NV-PJ3410_SOCKET_MONO" H 1950 2500 50  0001 C CNN
-F 3 "~" H 1950 2500 50  0001 C CNN
-	1    1950 2500
-	1    0    0    1
-$EndComp
-$Comp
-L Connector:AudioJack2_Ground J2
-U 1 1 5BCF798F
-P 9400 2500
-F 0 "J2" H 9167 2479 50  0000 R CNN
-F 1 "AudioJack2_Ground" H 9167 2570 50  0000 R CNN
-F 2 "MusicThingModular:NV-PJ3410_SOCKET_MONO" H 9400 2500 50  0001 C CNN
-F 3 "~" H 9400 2500 50  0001 C CNN
-	1    9400 2500
-	-1   0    0    1
-$EndComp
 $Comp
 L Device:C C2
@@
 F 0 "R1" H 3120 2946 50  0000 L CNN
 F 1 "R" H 3120 2855 50  0000 L CNN
-F 2 "MusicThingModular:10MM_RESISTOR" V 2980 2900 50  0001 C CNN
+F 2 "Resistor_THT:R_Axial_DIN0207_L6.3mm_D2.5mm_P10.16mm_Horizontal" V 2980 2900 50  0001 C CNN
 F 3 "~" H 3050 2900 50  0001 C CNN
 	1    3050 2900
@@
 F 0 "R2" H 4220 2946 50  0000 L CNN
 F 1 "R" H 4220 2855 50  0000 L CNN
-F 2 "MusicThingModular:10MM_RESISTOR" V 4080 2900 50  0001 C CNN
+F 2 "Resistor_THT:R_Axial_DIN0207_L6.3mm_D2.5mm_P10.16mm_Horizontal" V 4080 2900 50  0001 C CNN
 F 3 "~" H 4150 2900 50  0001 C CNN
 	1    4150 2900
@@
 F 0 "R3" V 4293 2500 50  0000 C CNN
 F 1 "R" V 4384 2500 50  0000 C CNN
-F 2 "MusicThingModular:10MM_RESISTOR" V 4430 2500 50  0001 C CNN
+F 2 "Resistor_THT:R_Axial_DIN0207_L6.3mm_D2.5mm_P10.16mm_Horizontal" V 4430 2500 50  0001 C CNN
 F 3 "~" H 4500 2500 50  0001 C CNN
 	1    4500 2500
@@
 F 0 "R4" H 4920 2946 50  0000 L CNN
 F 1 "R" H 4920 2855 50  0000 L CNN
-F 2 "MusicThingModular:10MM_RESISTOR" V 4780 2900 50  0001 C CNN
+F 2 "Resistor_THT:R_Axial_DIN0207_L6.3mm_D2.5mm_P10.16mm_Horizontal" V 4780 2900 50  0001 C CNN
 F 3 "~" H 4850 2900 50  0001 C CNN
 	1    4850 2900
@@
 F 0 "R5" V 8143 2500 50  0000 C CNN
 F 1 "R" V 8234 2500 50  0000 C CNN
-F 2 "MusicThingModular:10MM_RESISTOR" V 8280 2500 50  0001 C CNN
+F 2 "Resistor_THT:R_Axial_DIN0207_L6.3mm_D2.5mm_P10.16mm_Horizontal" V 8280 2500 50  0001 C CNN
 F 3 "~" H 8350 2500 50  0001 C CNN
 	1    8350 2500
@@
 Text Notes 2250 6550 0    50   ~ 0
 Inductors at Mouser: \nC-1X    15H (Triad Magnetics)\nC-85X  1.5H (Triad Magnetics)
+NoConn ~ 9200 2400
+NoConn ~ 2150 2400
+$Comp
+L hakane:AudioJack_Mono_Switch J1
+U 1 1 5C5B0CA6
+P 1950 2500
+F 0 "J1" H 1717 2479 50  0000 R CNN
+F 1 "TRIG_IN" H 1717 2570 50  0000 R CNN
+F 2 "kicadlib:PJ301BM" H 1950 2500 50  0001 C CNN
+F 3 "~" H 1950 2500 50  0001 C CNN
+	1    1950 2500
+	1    0    0    1
+$EndComp
+$Comp
+L hakane:AudioJack_Mono_Switch J2
+U 1 1 5C5B0D0D
+P 9400 2500
+F 0 "J2" H 9167 2479 50  0000 R CNN
+F 1 "AUDIO_OUT" H 9167 2570 50  0000 R CNN
+F 2 "kicadlib:PJ301BM" H 9400 2500 50  0001 C CNN
+F 3 "~" H 9400 2500 50  0001 C CNN
+	1    9400 2500
+	-1   0    0    1
+$EndComp
 $EndSCHEMATC

Commit message: Polish up the DR-77/78 schematic
Parts:
- removed JP1: ALT_COIL, Connector_PinHeader_2.54mm:PinHeader_1x03_P2.54mm_Vertical, symbol Jumper:Jumper_3_Bridged12
- added JP1: DARK_POT, Connector_PinHeader_2.54mm:PinHeader_1x02_P2.54mm_Vertical, symbol Device:Jumper_NC_Small
- added L2: (no value), Inductor_THT:L_Radial_D10.0mm_P5.00mm_Fastron_07P, symbol Device:L
- added SW1: ALT_COIL, Connector_PinHeader_2.54mm:PinHeader_1x03_P2.54mm_Vertical, symbol Switch:SW_SPDT
- C1, C10, C2, C3, C4, C5, C6, C7, C8, C9: value C -> (none)
- D1: value D -> (none)
- L1: value L -> (none)
- R1, R2, R3, R4, R5: value R -> (none)
Connections:
- wire segments 58 -> 62
- no-connect marks 3 -> 2
Other:
- note added: "JP1 can be used to connect a\nvariable resistance, for an option\nfor a darker sound. Just solder a\njumper if that’s not wanted."
- note added: "SW1/L2 can be used to add an extra coil, \nto be able to switch between sounds (higher\nor lower frequency). If not wanted, skip J2, \nand put a jumper between 1-2 on SW1."
- note added: "This schematic/PCB is far more complicated than it is, simply because \nI wanted the option to build several different sounds. A consequence \nof that is that several components must be left unmounted (”N/A”), or\nin some cases replaced with a piece of wire (”jumper”)."
- note removed: "JP1 can be used to connect a\ndifferent coil, e.g. via external jack."

Commit message: Clean up, and finish PCB
Removing the worst of the switch excesses (or adding a few switches,
depending on what was in the last commit).
Parts:
- removed JP1: DARK_POT, Connector_PinHeader_2.54mm:PinHeader_1x02_P2.54mm_Vertical, symbol Device:Jumper_NC_Small
- removed R5: (no value), Resistor_THT:R_Axial_DIN0207_L6.3mm_D2.5mm_P10.16mm_Horizontal, symbol Device:R
- removed SW1: ALT_COIL, Connector_PinHeader_2.54mm:PinHeader_1x03_P2.54mm_Vertical, symbol Switch:SW_SPDT
- added C11: (no value), Capacitor_THT:C_Rect_L7.2mm_W2.5mm_P5.00mm_FKS2_FKP2_MKS2_MKP2, symbol Device:C
- added D2: LED_ALT, LED_THT:LED_D3.0mm, symbol Device:LED_ALT
- added J3: EXT_COIL, kicadlib:PJ301BM, symbol hakane:AudioJack_Mono_Switch
- added R5: CUTOFF, Potentiometer_THT:Potentiometer_Alps_RK09K_Single_Vertical, symbol Device:R_POT
- added R6: (no value), Resistor_THT:R_Axial_DIN0207_L6.3mm_D2.5mm_P10.16mm_Horizontal, symbol Device:R
- added SW1: LPF/HPF_IN, kicadlib:DPDT_PUSH_SW, symbol Switch:SW_DPDT_x2
- added SW2: RS/C, kicadlib:DPDT_PUSH_SW, symbol Switch:SW_DPDT_x2
- added SW3: C6_SEL, kicadlib:DPDT_AS_SPST_PUSH_SW, symbol Switch:SW_SPST
- added SW4: COIL_1, kicadlib:DPDT_AS_SPST_PUSH_SW, symbol Switch:SW_SPST
- added SW5: COIL_2, kicadlib:DPDT_AS_SPST_PUSH_SW, symbol Switch:SW_SPST
- added SW6: C11_SEL, kicadlib:DPDT_AS_SPST_PUSH_SW, symbol Switch:SW_SPST
- added SW7: C8_SEL, kicadlib:DPDT_AS_SPST_PUSH_SW, symbol Switch:SW_SPST
- added SW8: STR_OUT, kicadlib:DPDT_AS_SPST_PUSH_SW, symbol Switch:SW_SPST
- added SW9: LPF/HPF_OUT, kicadlib:DPDT_PUSH_SW, symbol Switch:SW_DPDT_x2
- added TP1, TP2, TP3, TP4, TP5, TP6: (no value), TestPoint:TestPoint_THTPad_2.0x2.0mm_Drill1.0mm, symbol Connector:TestPoint
- added TP7: DEFAULT_EXT_COIL, TestPoint:TestPoint_THTPad_2.0x2.0mm_Drill1.0mm, symbol Connector:TestPoint
Connections:
- wire segments 62 -> 108
Other:
- note added: "(*) The diode is most likely not that important.\nI think I’ll go for a BAT-42, since it has low voltage\ndrop; I’m sure a standard 1N4148 will do as well."
- note added: "April 9, 2019"
- note added: "CR-78 Claves\n—————————\nC1: 27nF\nR1: 270k\nC2: NC\nD1: 1S1588 (*)\nR2: 2.2M\nR3: 47k\nR4: NC\nC3: 4.7 nF\nC4: 2.2 nF\nC5: 4.7 nF\nC6: NC\nL1: 700 mH\nC7: 250 pF\nC8: 5.6 nF\nC9: 1 nF\nR5: NC\nC10: NC\n"
- note added: "CR-78 Rim Shot\n—————————\nC1: 27nF\nR1: 270k\nC2: NC\nD1: 1S1588 (*)\nR2: NC\nR3: 47k\nR4: 47k\nC3: NC\nC4: 0 (jumper)\nC5: 1.5 nF\nC6: 15 nF\nL1: 700 mH\nC7: 470 pF\nC8: NC\nC9: NC\nR5: 0 (jumper)\nC10: NC"
- note added: "NOTE: R5 is a fixed resistor in TR-77’s BD, but a pot of\napprox. 20-50k might be useful as a variable LPF (untested)."
- note added: "NOTE: The LED will probably take a bit of the sound (amplitude, at \nleast). I included it on the PCB anyway, try with a low power LED and\na high resistor if you want a flashing LED – or just skip them if you \nwant to max the output."
- note added: "TR-77 Bass Drum\n—————————\nC1: 0 (jumper)\nR1: NC\nC2: 4.7 nF\nD1: 1S1555 (*)\nR2: 4.7M\nR3: 33k\nR4: NC\nC3: 56 nF\nC4: 33 nF\nC5: 220 nF\nC6: 1 nF\nL1: 16 H (!)\nC7: 33 nF\nC8: 100 nF\nC9: NC\nR5: 10 k\nC10: 220 nF"
- note added: "TR-77 Claves\n—————————\nC1: 0 (jumper)\nR1: NC\nC2: 4.7 nF\nD1: 1S1555 (*)\nR2: 4.7M\nR3: 56k\nR4: NC\nC3: 4.7 nF\nC4: 1 nF\nC5: 4.7 nF\nC6: NC\nL1: 700 mH\nC7: 1.5 nF\nC8: 5.6 nF\nC9: 2.2 nF\nR5: NC\nC10: NC"
- note added: "TR-77 Rim Shot\n—————————\nC1: 0 (jumper)\nR1: NC\nC2: 4.7 nF\nD1: 1S1555 (*)\nR2: 4.7M\nR3: 100k\nR4: 47k\nC3: NC\nC4: 0 (jumper)\nC5: 27 nF\nC6: NC\nL1: 700 mH\nC7: 1 nF\nC8: NC\nC9: NC\nR5: 0 (jumper)\nC10: NC\n"
- note added: "This schematic/PCB seems far more complicated than it is, simply because \nI wanted the option to build several different sounds, like a prototype.\nIf you want to build just one sound, check the table and figure out\nwhich components to leave out, and which pads on the switches that \nneeds to be shorted with jumpers (i.e., in that case, you don’t need\nthe switches).\nIf you want to change the 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"
- note removed: "CR-78 Claves\n—————————\nC1: 27nF\nR1: 270k\nC2: NC\nD1: (see note)\nR2: 2.2M\nR3: 47k\nR4: NC\nC3: 4.7 nF\nC4: 2.2 nF\nC5: 4.7 nF\nC6: NC\nL1: 700 mH\nC7: 250 pF\nC8: 5.6 nF\nC9: 1 nF\nR5: NC\nC10: NC\n"
- note removed: "CR-78 Rim Shot\n—————————\nC1: 27nF\nR1: 270k\nC2: NC\nD1: (see note)\nR2: NC\nR3: 47k\nR4: 47k\nC3: NC\nC4: NC\nC5: 1.5 nF\nC6: 15 nF\nL1: 700 mH\nC7: 470 pF\nC8: NC\nC9: NC\nR5: 0 (jumper)\nC10: NC"
- note removed: "JP1 can be used to connect a\nvariable resistance, for an option\nfor a darker sound. Just solder a\njumper if that’s not wanted."
- note removed: "January 26, 2019"
- note removed: "NOTE: For C1 on the TR-77 sounds: instead of a jumper,\ntry 27nF as on the CR-78 – is there a difference?"
- note removed: "NOTE: The diode is most likely not that important.\nI think I’ll go for a BAT-42, since it has low voltage\ndrop; I’m sure a standard 1N4148 will do as well.\nIf you want the original, check the original schematics. :-)"
- note removed: "SW1/L2 can be used to add an extra coil, \nto be able to switch between sounds (higher\nor lower frequency). If not wanted, skip J2, \nand put a jumper between 1-2 on SW1."
- note removed: "TR-77 Bass Drum\n—————————\nC1: 0 (jumper)\nR1: NC\nC2: 4.7 nF\nD1: (see note)\nR2: 4.7M\nR3: 33k\nR4: NC\nC3: 56 nF\nC4: 33 nF\nC5: 220 nF\nC6: 1 nF\nL1: 16 H (!)\nC7: 33 nF\nC8: 100 nF\nC9: NC\nR5: 10 k\nC10: 220 nF"
- note removed: "TR-77 Claves\n—————————\nC1: 0 (jumper)\nR1: NC\nC2: 4.7 nF\nD1: (see note)\nR2: 4.7M\nR3: 56k\nR4: NC\nC3: 4.7 nF\nC4: 1 nF\nC5: 4.7 nF\nC6: NC\nL1: 700 mH\nC7: 1.5 nF\nC8: 5.6 nF\nC9: 2.2 nF\nR5: NC\nC10: NC"
- note removed: "TR-77 Rim Shot\n—————————\nC1: 0 (jumper)\nR1: NC\nC2: 4.7 nF\nD1: (see note)\nR2: 4.7M\nR3: 100k\nR4: 47k\nC3: NC\nC4: 0 (jumper)\nC5: 27 nF\nC6: NC\nL1: 700 mH\nC7: 1 nF\nC8: NC\nC9: NC\nR5: 0 (jumper)\nC10: NC\n"
- note removed: "This schematic/PCB is far more complicated than it is, simply because \nI wanted the option to build several different sounds. A consequence \nof that is that several components must be left unmounted (”N/A”), or\nin some cases replaced with a piece of wire (”jumper”)."
