File: minidrum-77/kicad_files/minidrum-77.sch (KiCad schematic (older format))
At the start: 40 parts, among them J1 TRIG_IN, J2 AUDIO_OUT, J3 EXT_COIL, SW1 LPF/HPF_IN, SW2 RS/C, SW3 C6_SEL, SW4 COIL_1, SW5 COIL_2, SW6 C11_SEL, SW7 C8_SEL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

Commit message: minidrum: Move switches apart a bit
Experiments with PCB layout on paper indicated that the
space between switches was too tight. Maybe still, but better.

Also cleaning up other PCBs a bit.
Parts:
- removed TP1, TP2, TP6: (no value), TestPoint:TestPoint_THTPad_2.0x2.0mm_Drill1.0mm, symbol Connector:TestPoint
- removed TP7: DEFAULT_EXT_COIL, TestPoint:TestPoint_THTPad_2.0x2.0mm_Drill1.0mm, symbol Connector:TestPoint
- renumbered TP3 to TP1, TP4 to TP2, TP5 to TP3
Connections:
- wire segments 108 -> 103
- no-connect marks 2 -> 3
Changed lines of the file:
@@
 	9800 2750 10150 2750
-Wire Wire Line
-	3300 2100 3300 2750
 Wire Wire Line
 	6900 2850 6900 2950
@@
 Wire Wire Line
 	6100 2100 6100 2850
-$Comp
-L Connector:TestPoint TP1
-U 1 1 5CAF128C
-P 1500 2100
-F 0 "TP1" H 1558 2220 50  0000 L CNN
-F 1 " " H 1558 2129 50  0000 L CNN
-F 2 "TestPoint:TestPoint_THTPad_2.0x2.0mm_Drill1.0mm" H 1700 2100 50  0001 C CNN
-F 3 "~" H 1700 2100 50  0001 C CNN
-	1    1500 2100
-	1    0    0    -1
-$EndComp
-Wire Wire Line
-	1500 2100 1500 2650
 Wire Wire Line
 	8350 2100 8350 2350
@@
 	8350 2350 8350 2850
 $Comp
-L Connector:TestPoint TP6
-U 1 1 5CB0E70E
-P 10600 2100
-F 0 "TP6" H 10658 2220 50  0000 L CNN
-F 1 " " H 10658 2129 50  0000 L CNN
-F 2 "TestPoint:TestPoint_THTPad_2.0x2.0mm_Drill1.0mm" H 10800 2100 50  0001 C CNN
-F 3 "~" H 10800 2100 50  0001 C CNN
-	1    10600 2100
-	1    0    0    -1
-$EndComp
-Wire Wire Line
-	10600 2100 10600 2250
-Connection ~ 10600 2250
-$Comp
-L Connector:TestPoint TP5
+L Connector:TestPoint TP3
 U 1 1 5CB23654
 P 8350 2100
-F 0 "TP5" H 8408 2220 50  0000 L CNN
+F 0 "TP3" H 8408 2220 50  0000 L CNN
 F 1 " " H 8408 2129 50  0000 L CNN
 F 2 "TestPoint:TestPoint_THTPad_2.0x2.0mm_Drill1.0mm" H 8550 2100 50  0001 C CNN
@@
 $EndComp
 $Comp
-L Connector:TestPoint TP4
+L Connector:TestPoint TP2
 U 1 1 5CB236D5
 P 6100 2100
-F 0 "TP4" H 6158 2220 50  0000 L CNN
+F 0 "TP2" H 6158 2220 50  0000 L CNN
 F 1 " " H 6158 2129 50  0000 L CNN
 F 2 "TestPoint:TestPoint_THTPad_2.0x2.0mm_Drill1.0mm" H 6300 2100 50  0001 C CNN
@@
 $EndComp
 $Comp
-L Connector:TestPoint TP3
+L Connector:TestPoint TP1
 U 1 1 5CB2375A
 P 4100 2100
-F 0 "TP3" H 4158 2220 50  0000 L CNN
+F 0 "TP1" H 4158 2220 50  0000 L CNN
 F 1 " " H 4158 2129 50  0000 L CNN
 F 2 "TestPoint:TestPoint_THTPad_2.0x2.0mm_Drill1.0mm" H 4300 2100 50  0001 C CNN
 F 3 "~" H 4300 2100 50  0001 C CNN
 	1    4100 2100
-	1    0    0    -1
-$EndComp
-$Comp
-L Connector:TestPoint TP2
-U 1 1 5CB237D7
-P 3300 2100
-F 0 "TP2" H 3358 2220 50  0000 L CNN
-F 1 " " H 3358 2129 50  0000 L CNN
-F 2 "TestPoint:TestPoint_THTPad_2.0x2.0mm_Drill1.0mm" H 3500 2100 50  0001 C CNN
-F 3 "~" H 3500 2100 50  0001 C CNN
-	1    3300 2100
 	1    0    0    -1
 $EndComp
@@
 Wire Wire Line
 	9850 2950 9950 2950
-$Comp
-L Connector:TestPoint TP7
-U 1 1 5CA968CB
-P 7450 4200
-F 0 "TP7" H 7500 4350 50  0000 L CNN
-F 1 "DEFAULT_EXT_COIL" H 7600 4300 50  0000 L CNN
-F 2 "TestPoint:TestPoint_THTPad_2.0x2.0mm_Drill1.0mm" H 7650 4200 50  0001 C CNN
-F 3 "~" H 7650 4200 50  0001 C CNN
-	1    7450 4200
-	1    0    0    -1
-$EndComp
-Wire Wire Line
-	7450 4200 7450 4250
-Wire Wire Line
-	7450 4250 7500 4250
 Wire Wire Line
 	7350 4350 7500 4350
@@
 Text Notes 1350 1600 0    59   ~ 0
 NOTE: The LED will probably take a bit of the sound (amplitude, at \nleast). I included it on the PCB anyway, try with a low power LED and\na high resistor if you want a flashing LED – or just skip them if you \nwant to max the output.
+NoConn ~ 7500 4250
 $EndSCHEMATC

Commit message: Just notes in some schematics
Parts:
- R6: value (none) -> 4.7k
Other:
- note added: "Inductors of such large values are hard to find. \nThe PCB is made for the following two, available \nfrom Mouser: \nC-1X 15H (Triad Magnetics)\nC-85X 1.5H (Triad Magnetics)"
- note added: "NOTE: C1/R1 and/or C2 might be useless. Experiment."
- note added: "NOTE: C9 is pretty stupid, taken out of context as it it. Its HPF \nproperties depend on what comes after. Maybe it’d be more interesting \nto turn the LPF around? Far from the original, but still."
- note added: "NOTE: Should have had a switch for C3/C4, since their values differ so much."
- note added: "NOTE: The LED will probably take a bit of the sound (amplitude, at \nleast). I included it on the PCB anyway, try with a low power LED and\na high resistor if you want a flashing LED – or just skip them if you \nwant to max the output.\nAdjust R6 to your liking (and the LED’s max current)."
- note added: "NOTE: The components listed are (pretty much) taken from the \nschematics of these machines. When building it might make sense to\nad lib a bit, for instance: C5/C6 are used in a couple of sounds to fine\ntune the resonance frequency (I guess) – another option is to choose\nvalues of greater difference, for larger sonic tweakability (if you do: put \nthe larger values on the switches). Let your e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"
- note removed: "Inductors at Mouser: \nC-1X 15H (Triad Magnetics)\nC-85X 1.5H (Triad Magnetics)"
- note removed: "NOTE: The LED will probably take a bit of the sound (amplitude, at \nleast). I included it on the PCB anyway, try with a low power LED and\na high resistor if you want a flashing LED – or just skip them if you \nwant to max the output."
Changed lines of the file:
@@
 Text Notes 5700 6200 0    59   ~ 0
 TR-77 Bass Drum\n—————————\nC1: 0 (jumper)\nR1: NC\nC2: 4.7 nF\nD1: 1S1555 (*)\nR2: 4.7M\nR3: 33k\nR4: NC\nC3: 56 nF\nC4: 33 nF\nC5: 220 nF\nC6: 1 nF\nL1: 16 H (!)\nC7: 33 nF\nC8: 100 nF\nC9: NC\nR5: 10 k\nC10: 220 nF
-Text Notes 3900 6850 0    59   ~ 0
+Text Notes 3500 7150 0    59   ~ 0
 NOTE: R5 is a fixed resistor in TR-77’s BD, but a pot of\napprox. 20-50k might be useful as a variable LPF (untested).
 Wire Wire Line
@@
 Text Notes 10650 7650 0    50   ~ 0
 A
-Text Notes 3900 7150 0    59   ~ 0
+Text Notes 3500 7400 0    59   ~ 0
 NOTE: The coil values for the listed CR-78 voices are guessed:\nhttp://electro-music.com/forum/post-420004.html#420004
-Text Notes 3900 7500 0    59   ~ 0
+Text Notes 3500 7750 0    59   ~ 0
 (*) The diode is most likely not that important.\nI think I’ll go for a BAT-42, since it has low voltage\ndrop; I’m sure a standard 1N4148 will do as well.
-Text Notes 2100 7300 0    50   ~ 0
-Inductors at Mouser: \nC-1X    15H (Triad Magnetics)\nC-85X  1.5H (Triad Magnetics)
+Text Notes 1000 6800 0    59   ~ 0
+Inductors of such large values are hard to find. \nThe PCB is made for the following two, available \nfrom Mouser: \nC-1X    15H (Triad Magnetics)\nC-85X  1.5H (Triad Magnetics)
 NoConn ~ 10650 2750
 NoConn ~ 1250 2650
@@
 Connection ~ 6900 3950
 Text Notes 7400 6350 0    59   ~ 0
-This schematic/PCB seems far more complicated than it is, simply because \nI wanted the option to build several different sounds, like a prototype.\nIf you want to build just one sound, check the table and figure out\nwhich components to leave out, and which pads on the switches that \nneeds to be shorted with jumpers (i.e., in that case, you don’t need\nthe switches).\nIf you want to change the sound somewhat, go all in with the switches \nand stuff. Note that it’s probably impossible to get two authentic \noriginal sounds, as the exact component values vary, but you can \nget one actual sound, and then experiment to get something else \nwith the switches.
+This schematic/PCB seems far more complicated than it is, simply because \nI wanted the option to build several different sounds, like a prototype.\nIf you want to build just one sound, check the table and figure out\nwhich components to leave out, and which pads on the switches that \nneeds to be shorted with jumpers (i.e., in that case, you don’t need\nthe switches).\nIf you want to change the sound somewhat, go all in with the switches \nand stuff. Note that it’s impossible to get two authentic original sounds, \nas the exact component values vary, plus that I didn’t think enough \nahead,but you can get one actual sound, and then experiment to get \nsomething else with the switches.
 Wire Wire Line
 	6600 2850 6900 2850
@@
 P 1500 3550
 F 0 "R6" H 1600 3600 50  0000 L CNN
-F 1 " " H 1570 3505 50  0000 L CNN
+F 1 "4.7k" H 1570 3505 50  0000 L CNN
 F 2 "Resistor_THT:R_Axial_DIN0207_L6.3mm_D2.5mm_P10.16mm_Horizontal" V 1430 3550 50  0001 C CNN
 F 3 "~" H 1500 3550 50  0001 C CNN
@@
 	6900 4450 7500 4450
 Text Notes 1350 1600 0    59   ~ 0
-NOTE: The LED will probably take a bit of the sound (amplitude, at \nleast). I included it on the PCB anyway, try with a low power LED and\na high resistor if you want a flashing LED – or just skip them if you \nwant to max the output.
+NOTE: The LED will probably take a bit of the sound (amplitude, at \nleast). I included it on the PCB anyway, try with a low power LED and\na high resistor if you want a flashing LED – or just skip them if you \nwant to max the output.\nAdjust R6 to your liking (and the LED’s max current).
 NoConn ~ 7500 4250
+Text Notes 3500 6900 0    59   ~ 0
+NOTE: The components listed are (pretty much) taken from the \nschematics of these machines. When building it might make sense to\nad lib a bit, for instance: C5/C6 are used in a couple of sounds to fine\ntune the resonance frequency (I guess) – another option is to choose\nvalues of greater difference, for larger sonic tweakability (if you do: put \nthe larger values on the switches). Let your ears and hearts decide.
+Text Notes 1350 1850 0    59   ~ 0
+NOTE: Should have had a switch for C3/C4, since their values differ so much.
+Text Notes 7650 1750 0    59   ~ 0
+NOTE: C9 is pretty stupid, taken out of context as it it. Its HPF \nproperties depend on what comes after. Maybe it’d be more interesting \nto turn the LPF around? Far from the original, but still.
+Text Notes 1350 1050 0    59   ~ 0
+NOTE: C1/R1 and/or C2 might be useless. Experiment.
 $EndSCHEMATC

Commit message: Add info on my minidrum implementation, my values
Other:
- note added: "My pick\nR6: 4.7k for a 2mA red LED\nC1: 22nF\nR1: 270k\nC2: 68nF\nD1: BAT42\nR2: 3.3M\nR3: 33k\nR4: 47k\nC3: 33//22 nF (~56nF)\nC4: 1nF (will evaluate, maybe larger)\nC6: 220nF (BD’s C5)\nC5: 1.5 nF\nL1: 15H\nL2: 120mH\nC11: 33nF (BD’s C7)\nC7: 1nF (TESTA 10nF)\nC8: 100nF\nC9: 10nF (SJHDFJHSDGFJHSGD)\nR5: 25k lin\nC10: 220nF"
Changed lines of the file:
@@
 Text Notes 1350 1050 0    59   ~ 0
 NOTE: C1/R1 and/or C2 might be useless. Experiment.
+Text Notes 5300 2600 0    59   ~ 0
+My pick\nR6: 4.7k for a 2mA red LED\nC1: 22nF\nR1: 270k\nC2: 68nF\nD1: BAT42\nR2: 3.3M\nR3: 33k\nR4: 47k\nC3: 33//22 nF (~56nF)\nC4: 1nF (will evaluate, maybe larger)\nC6: 220nF (BD’s C5)\nC5: 1.5 nF\nL1: 15H\nL2: 120mH\nC11: 33nF (BD’s C7)\nC7: 1nF (TESTA 10nF)\nC8: 100nF\nC9: 10nF (SJHDFJHSDGFJHSGD)\nR5: 25k lin\nC10: 220nF
 $EndSCHEMATC
