File: 4xvca/kicad_files/4xvca.sch (KiCad schematic (older format))
At the start: 101 parts, among them J1 CV_1, J10 OUT_1, J11 OUT_2, J12 OUT_3, J13 OUT_4, J14 MIX_OUT, J2 CV_2, J3 CV_3, J4 CV_4, J5 EUROPOWER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

Commit message: Unknown changes in 4xVCA (yes, unknown)
Parts:
- removed R21, R22, R23, R24, R25, R26, R27, R28: 100k, Resistors_THT:R_Axial_DIN0207_L6.3mm_D2.5mm_P7.62mm_Horizontal, symbol 4xvca-rescue:R
- removed R55: 1k, Resistors_THT:R_Axial_DIN0207_L6.3mm_D2.5mm_P7.62mm_Horizontal, symbol 4xvca-rescue:R
- removed R56: 100, Resistors_THT:R_Axial_DIN0207_L6.3mm_D2.5mm_P7.62mm_Horizontal, symbol 4xvca-rescue:R
- removed U2: TL074, Housings_DIP:DIP-14_W7.62mm_Socket_LongPads, symbol 4xvca-rescue:TL074
- removed U5: TL071, Housings_DIP:DIP-8_W7.62mm_Socket_LongPads, symbol 4xvca-rescue:TL071
- added C? (x2): 100nF, Capacitors_THT:C_Rect_L7.2mm_W3.5mm_P5.00mm_FKS2_FKP2_MKS2_MKP2, symbol 4xvca-rescue:C
- added D3: BAT41, symbol Device:D_Schottky
- added R? (x2): 100k, Resistors_THT:R_Axial_DIN0207_L6.3mm_D2.5mm_P7.62mm_Horizontal, symbol 4xvca-rescue:R
- added R?: 1k, Resistors_THT:R_Axial_DIN0207_L6.3mm_D2.5mm_P7.62mm_Horizontal, symbol 4xvca-rescue:R
- added R?: 100, Resistors_THT:R_Axial_DIN0207_L6.3mm_D2.5mm_P7.62mm_Horizontal, symbol 4xvca-rescue:R
- added U? (x3): TL072, symbol Amplifier_Operational:TL072
- R54: value 100k -> 22k
Connections:
- wire segments 290 -> 294
- no-connect marks 2 -> 0
Other:
- note added: "MAJOR TODO: \nJust found a document mentioning that the VCA control is exponential, \nand a schematic that uses two of the VCAs to make it linear (and a way \nto switch between the two). \nImplement that. A lot more boring to take someone’s schematic, and a \npity to lose two VCAs, but I read that linear is more normal in synths.\n\nhttp://www.sdiy.org/philgallo/mgbvca.html"
- note added: "Straight out of the VS2164 (or SSM2164) data sheet, a basic VCA. \nAdded a mix output.\nThe Schottky diode is to protect the IC, see: \nhttp://www.muffwiggler.com/forum/viewtopic.php?t=96486"
- note removed: "Straight out of the VS2164 (or SSM2164) data sheet, \na really basic VCA, no frills."
- moved on the sheet: C1, C10, C2, C3, C4, C5, C6, C7, C8, C9, D1, D2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
